File: LTC3105/main.sch (EAGLE design)
At the start: 13 parts

Commit message: updated project
Parts:
- added GND@0, GND@1, GND@2, OUTLDO: (no value), 7_segment_lib:2,54/1,0
- C2: device eagle-ltspice:CC0603 -> rcl:C-US025-025X050
- C3, C4: device rcl:CPOL-USE2-5 -> rcl:CPOL-USE1.8-4
- C5, C6: device rcl:CPOL-USE3.5-8 -> rcl:CPOL-USE2-5
- IN, OUT: device wirepad:SMD2 -> 7_segment_lib:2,54/1,0
- R1: device rcl:R-US_0204/7 -> rcl:R-US_0204/2V
- R2: device rcl:R-US_0309/V -> rcl:R-US_R0603
Connections:
- net GND: now also GND@0.P, GND@1.P, GND@2.P
- net N$2: now also OUTLDO.P
