File: 32u4/main.sch (EAGLE design)
At the start: 15 parts, among them U1 ATMEGA32U4-TQFP44, X1 MINI-USB-UX60A-MB-5ST

Commit message: sdfsdfsff
Parts:
- removed SV1: (no value), con-lstb:MA08-1
- added C1: 100n, rcl:C-EUC0402
- added SV4: (no value), con-lstb:MA09-1
- added SW1: TL3330, 7_segment_lib:TL3330
- X1: value MINI-USB-UX60A-MB-5ST -> MINI-USB-SCHIELD-32005-201; device con-hirose:MINI-USB-UX60A-MB-5ST -> con-cypressindustries:MINI-USB-SCHIELD-32005-201
Connections:
- removed net 2A: SV2.1, U1.PE6(INT.6/AIN0)
- new net N$25: SV4.7, U1.PC6(OC3A/!OC4A)
- new net N$26: SV4.8, U1.PC7(ICP3/CLK0/OC4A)
- new net N$27: SV4.9, U1.PE2(!HWB)
- net GND: now also C1.1, R2.2, SV2.1, SW1.S1, SW1.SHIELD@0, SW1.SHIELD@1, X1G$1.5, X1S.S1, X1S.S2, X1S.S3, X1S.S4; no longer X1.5
- net LED: now also U1.PE6(INT.6/AIN0)
- net N$10: now also X1G$1.2; no longer X1.2
- net N$11: now also X1G$1.3; no longer X1.3
- net N$19: now also SV4.1; no longer SV1.1
- net N$20: now also SV4.2; no longer SV1.2
- net N$21: now also SV4.3; no longer SV1.3
- net N$22: now also SV4.4; no longer SV1.4
- net N$23: now also SV4.5; no longer SV1.5
- net N$24: now also SV4.6; no longer SV1.6
- net RST: now also SW1.S2
- net VCC: now also C1.2, X1G$1.1; no longer R2.2, X1.1
