File: AD5932/main.sch (EAGLE design)
At the start: 0 parts

Commit message: updated project
Parts:
- added C1, C2, C3, C4: 100n, rcl:C-USC0603
- added C5, C6: 10p, rcl:C-USC0603
- added Q1: 16MHz, crystal:CRYSTALHC49U-V
- added QG1: 40MHz, crystal:QG5460
- added SV1: (no value), con-lstb:MA06-1
- added U1: AD5932YRUZ, Analog Devices_By_element14_Batch_1:AD5932YRUZ
- added U2: ATMEGA32U4-AU, Atmel_By_element14_Batch_1-00:ATMEGA32U4-AU
- added X1: MINI-USB-32005-201, con-cypressindustries:MINI-USB-32005-201
Connections:
- new net GND: C1.2, C2.2, C3.2, C4.2, C5.2, C6.2, QG1.GND, SV1.1, U1.AGND, U1.DGND, U2.GND, U2.GND_2, U2.GND_3, U2.GND_4, U2.UGND
- new net MISO: SV1.2
- new net MOSI: SV1.3
- new net N$1: QG1.OUT, U1.MCLK
- new net N$4: C5.1, Q1.1, U2.XTAL2
- new net RESET: SV1.4
- new net SCK: SV1.5
- new net VCC: C1.1, C2.1, C3.1, C4.1, QG1.VCC, SV1.6, U1.AVDD, U1.DVDD, U2.AVCC, U2.AVCC_2, U2.UVCC, U2.VCC, U2.VCC_2
- new net XTAL1: C6.1, Q1.2, U2.XTAL1
