File: solar/main.brd (EAGLE design)
At the start: 73.7 x 66 mm, 28 parts

Commit message: updated project
Parts:
- removed R5: (no value), resistor:R0603
- added R0: (no value), resistor:R0603
- R1: value (none) -> 1.2M
- R2: value (none) -> 300k
- R3: value (none) -> 470k
- R4: value (none) -> 200k
- moved R4 8.17 mm to (-1.08, 17.3), turned to 90 degrees
- moved R2 7.43 mm to (1.92, 24.1)
- moved R1 7.00 mm to (4.50, 23.3)
Connections:
- net GND: now also R0.1, R2.2, R4.1; no longer R1.1, R2.1, R5.2
- net N$10: now also R0.2; no longer R1.2
- net N$11: now also R4.2; no longer R2.2
- net N$13: now also R1.2, R2.1; no longer R4.2, R5.1
- net VCC: now also R1.1; no longer R4.1
