File: olimex_lcd/main2.sch (EAGLE design)
At the start: 0 parts

Commit message: jhg
Parts:
- added IC1: ATMEGA6490, 7_segment_lib:ATMEGA6490
- added LCD1: LCD_OLIMEXLCD_OLIMEX, 7_segment_lib:LCD_OLIMEXLCD_OLIMEX
- added SV1: isp, con-lstb:MA06-1
Connections:
- new net 1: IC1._SEG0_PA4, LCD1.1
- new net 10: IC1._PCINT17/SEG9_PH1, LCD1.10
- new net 11: IC1._PCINT16/SEG10_PH0, LCD1.11
- new net 12: IC1._SEG11_PC5, LCD1.12
- new net 13: IC1._SEG12_PC4, LCD1.13
- new net 14: IC1._SEG13_PC3, LCD1.14
- new net 15: IC1._SEG14_PC2, LCD1.15
- new net 16: IC1._SEG15_PC1, LCD1.16
- new net 17: IC1._SEG16_PC0, LCD1.17
- new net 18: IC1._SEG17_PG1, LCD1.18
- new net 19: IC1._SEG18_PG0, LCD1.19
- new net 2: IC1._SEG1_PA5, LCD1.2
- new net 20: IC1._SEG19_PD7, LCD1.20
- new net 21: IC1._SEG20_PD6, LCD1.21
- new net 22: IC1._SEG21_PD5, LCD1.22
- new net 23: IC1._SEG22_PD4, LCD1.23
- new net 24: IC1._SEG23_PD3, LCD1.24
- new net 25: IC1._SEG24_PD2, LCD1.25
- new net 26: IC1._INTO/SEG25_PD1, LCD1.26
- new net 27: IC1._ICP1/SEG26_PDO, LCD1.27
- new net 28: IC1._PCINT30/SEG27_PJ6, LCD1.28
- new net 29: IC1._PCINT29/SEG28_PJ5, LCD1.29
- new net 3: IC1._SEG2_PA6, LCD1.3
- new net 30: IC1._PCINT28/SEG29_PJ4, LCD1.30
- new net 31: IC1._PCINT27/SEG30_PJ3, LCD1.31
- new net 32: IC1._PCINT26/SEG31_PJ2, LCD1.32
- new net 33: IC1._TO/SEG32_PG4, LCD1.33
- new net 34: IC1._T1/SEG33_PG3, LCD1.34
- new net 35: LCD1.35
- new net 36: IC1._PCINT25/SEG34_PJ1, LCD1.36
- new net 37: IC1._PCINT24/SEG35_PJ0, LCD1.37
- new net 38: LCD1.38
- new net 39: LCD1.39
- new net 4: IC1._SEG3_PA7, LCD1.4
- new net 40: IC1._PCINT23/SEG36_PH7, LCD1.40
- new net 41: IC1._PCINT22/SEG37_PH6, LCD1.41
- new net 42: LCD1.42
- new net 43: IC1._PCINT21/SEG38_PH5, LCD1.43
- new net 44: IC1._PCINT20/SEG39_PH4, LCD1.44
- new net 5: IC1._SEG4_PG2, LCD1.5
- new net 5V: IC1.AREF, IC1.AVCC, IC1.VCC, IC1.VCC@1, IC1.VCC@2, SV1.5
- new net 6: IC1._SEG5_PC7, LCD1.6
- new net 7: IC1._SEG6_PC6, LCD1.7
- new net 8: IC1._PCINT19/SEG7_PH3, LCD1.8
- new net 9: IC1._PCINT18/SEG8_PH2, LCD1.9
- new net COM0: IC1._COMO_FAO, LCD1.COM0
- new net COM1: IC1._COM1_PA1, LCD1.COM1
- new net COM2: IC1._COM2_PA2, LCD1.COM2
- new net COM3: IC1._COM3_PA3, LCD1.COM3
- new net GND: IC1.AGND, IC1.GND, IC1.GND@1, IC1.GND@2, SV1.6
- new net LCDCAP: IC1.LCDCAP
- new net MISO: IC1._MISO/PCINT11_PB3, SV1.1
- new net MOSI: IC1._MOSI/PCINT10_PB2, SV1.2
- new net RESET: IC1.RESET/PG5, SV1.4
- new net RX: IC1._RXD/PCINT0_PE0
- new net SCK: IC1._SCK/PCINT9_PB1, SV1.3
- new net TX: IC1._TXD/PCINT1_PE1
- new net XTAL1: IC1._TOSC2_XTAL2
- new net XTAL2: IC1._TOSC1_XTAL1
- new net _0C2A/PCINT15_PB7: IC1._0C2A/PCINT15_PB7
- new net _ADC1_PF1: IC1._ADC1_PF1
- new net _ADC2_PF2: IC1._ADC2_PF2
- new net _ADC3_PF3: IC1._ADC3_PF3
- new net _ADC4/TCK_PF4: IC1._ADC4/TCK_PF4
- new net _ADC5/TMS_PF5: IC1._ADC5/TMS_PF5
- new net _ADC6/TDO_PF6: IC1._ADC6/TDO_PF6
- new net _ADC7/TDI_PF7: IC1._ADC7/TDI_PF7
- new net _ADCO_PFO: IC1._ADCO_PFO
- new net _AIN1/PCINT3_PE3: IC1._AIN1/PCINT3_PE3
- new net _CLKO/PCINT7_PE7: IC1._CLKO/PCINT7_PE7
- new net _DI/SDA/PCINT5_PE5: IC1._DI/SDA/PCINT5_PE5
- new net _DO/PCINT6_PE6: IC1._DO/PCINT6_PE6
- new net _OC0A/PCINT12_PB4: IC1._OC0A/PCINT12_PB4
- new net _OC1A/PCINT13_PB5: IC1._OC1A/PCINT13_PB5
- new net _OC1B/PCINT14_PB6: IC1._OC1B/PCINT14_PB6
- new net _SS/PCINT8_PB0: IC1._SS/PCINT8_PB0
- new net _USCK/SCL/PCINT4_PE4: IC1._USCK/SCL/PCINT4_PE4
- new net _XCK/AIN0/PCINT2_PE2: IC1._XCK/AIN0/PCINT2_PE2
