File: TicTacToe/main.sch (EAGLE design)
At the start: 23 parts, among them U1 AT90USB1286-AU, Y1 16MHz

Commit message: ttt
Parts:
- removed CN1: (no value), adafruit:USBMINIB
- removed Y1: 16MHz, SparkFun-Clocks:CRYSTAL-16MHZPTH-HC49US
- added D1: BAT54, diode:BAT54
- added J1: (no value), SparkFun-Connectors:JST_2MM_MALE
- added U$1: MIC94090, 7_segment_lib:MIC94090
- added X2: MINI-USB-SHIELD-UX60A-MB-5ST, con-hirose:MINI-USB-SHIELD-UX60A-MB-5ST
- C1, C2: value 10p -> 100n
Connections:
- removed net ID: CN1.ID
- removed net X1: C1.1, U1.XTAL1, Y1.1
- removed net X2: C2.1, U1.XTAL2, Y1.2
- new net N$3: J1.PAD2
- new net N$4: J1.PAD1
- new net PA6: U1.PA6
- new net PA7: U1.PA7
- new net PB0: U1.PB0
- new net PB1: U1.PB1
- new net PB2: U1.PB2
- new net PB3: U1.PB3
- new net PB4: U1.PB4
- new net PB5: U1.PB5
- new net PB6: U1.PB6
- new net PB7: U1.PB7
- new net PC3: U1.PC3
- new net PC4: U1.PC4
- new net PC5: U1.PC5
- new net PC6: U1.PC6
- new net PC7: U1.PC7
- new net PD3: U1.PD3
- new net PD4: U1.PD4
- new net PD5: U1.PD5
- new net PD6: U1.PD6
- new net PD7: U1.PD7
- new net PE0: U1.PE0
- new net PE1: U1.PE1
- new net PE2: U1.PE2
- new net PE3: U1.PE3
- new net PE4: U1.PE4
- new net PE5: U1.PE5
- new net PE6: U1.PE6
- new net PE7: U1.PE7
- new net PF0: U1.PF0
- new net PF1: U1.PF1
- new net PF2: U1.PF2
- new net PF3: U1.PF3
- new net PF4: U1.PF4
- new net PF5: U1.PF5
- new net PF6: U1.PF6
- new net PF7: U1.PF7
- new net UCAP: U1.UCAP
- new net USB: D1.A, U$1.EN, X2G$1.1
- new net VBAT: J1.+, U$1.VIN
- new net XTAL1: U1.XTAL1
- new net XTAL2: U1.XTAL2
- new net ~RESET: U1.~RESET
- net C1: now also U1.PD1; no longer U1.PB0
- net C2: now also U1.PD2; no longer U1.PB1
- net C3: now also U1.PD0; no longer U1.PB2
- net D_N: no longer CN1.D-
- net D_P: no longer CN1.D+
- net GND: now also J1.-, U$1.GND@0, U$1.GND@1, X2G$1.5; no longer CN1.GND
- net L11: now also L3.A2, U1.PC1; no longer L3.A1, U1.PC0
- net L12: now also L3.A1, U1.PC0; no longer L3.A2, U1.PC1
- net L1B: now also U1.PA2
- net L21: now also L6.A2, U1.PA1; no longer L6.A1, U1.PC2
- net L22: now also L6.A1, U1.PA0; no longer L6.A2, U1.PC3
- net L2B: now also U1.PA5
- net L31: now also L9.A2, U1.PA3; no longer L9.A1, U1.PC4
- net L32: now also L9.A1, U1.PA4; no longer L9.A2, U1.PC5
- net L3B: now also U1.PC2
- net VCC: now also C1.1, C2.1, D1.C, U$1.VOUT, U1.AREF; no longer CN1.VBUS
Other:
- moved on the sheet: C1, C2
