File: TicTacToe/main1.brd (EAGLE design)
At the start: 80 x 80 mm, 33 parts, among them U1 ATMEGA168-20AU, X2 MINI-USB-SHIELD-UX60A-MB-5ST

Commit message: updated project
Connections:
- removed net N$3: J1.NC2
- removed net N$4: J1.NC1
- new net N$1: J1.NC1, J1.NC2
Routing:
- added copper zone on layer 1, net GND
- added copper zone on layer 16, net N$1
