File: miliohmeter/main.sch (EAGLE design)
At the start: 39 parts, among them U1 LT6656ACS6-2.5PBF, U2 ATMEGA169P-16AU, X1 SMA-142-0701-801/806, X2 SMA-142-0701-801/806, X3 SMA-142-0701-801/806, X4 SMA-142-0701-801/806

Commit message: miliohmeter
Parts:
- removed U1: LT6656ACS6-2.5PBF, LTC_By_element14_Batch_1:LT6656ACS6-2.5PBF
- removed X1, X2, X3, X4: SMA-142-0701-801/806, con-coax:SMA-142-0701-801/806
- added C14, C15: 1u, rcl:C-USC0603
- added C16, C18: 100n, rcl:C-USC0603
- added IC1: LT1019S-2.5, linear-technology:LT1019S-2.5
- added LSP1, LSP2, LSP3, LSP4: MCS08, solpad:MCS08
- added R13, R15, R16: 1k, rcl:R-US_R0603
- added R14, R17, R18: 100, rcl:R-US_R0603
- added R19: 10k, rcl:R-US_R0603
- added S2: MOMENTARY-SWITCH-SPST-SMD-6.0X3.5MM, SparkFun-Switches:MOMENTARY-SWITCH-SPST-SMD-6.0X3.5MM
- added U3: MCP6V02-E/SN, Microchip_By_element14_Batch_1:MCP6V02-E/SN
- added USART: (no value), con-lstb:MA03-1
Connections:
- net N$1 renamed VFG
- removed net GND_2: U2.GND_2
- removed net GND_3: U2.GND_3
- removed net PD0: U2.PD0
- removed net PE0: U2.PE0
- removed net PE1: U2.PE1
- removed net PF4: U2.PF4
- removed net PF5: U2.PF5
- removed net SHIELD: X1.2, X2.2, X3.2, X4.2
- new net B2: C18.1, R16.1, R19.1, U2.PF5
- new net N$7: R13.2, U3.VOUTA
- new net N$8: R13.1, T1.B
- new net N$9: R15.1, U3.VINA-
- new net N2: R16.2, S2.1
- new net RX: U2.PE0, USART.2
- new net TX: U2.PE1, USART.3
- new net VOUT: R6.1, R8.2, U$3.VOUT
- new net VREF: R5.2, R7.2, U$3.VREF
- net 1: now also U$7.13; no longer U$7.1
- net 10: now also U$7.4; no longer U$7.10
- net 11: now also U$7.3; no longer U$7.11
- net 12: now also U$7.2; no longer U$7.12
- net 13: now also U$7.1; no longer U$7.13
- net 2: now also U$7.12; no longer U$7.2
- net 3: now also U$7.11; no longer U$7.3
- net 4: now also U$7.10; no longer U$7.4
- net 5: now also U$7.9; no longer U$7.5
- net 6: now also U$7.8; no longer U$7.6
- net 8: now also U$7.6; no longer U$7.8
- net 9: now also U$7.5; no longer U$7.9
- net GND: now also R19.2, U2.GND_2, U2.GND_3, USART.1
- net GNDA: now also C14.2, C15.2, C16.2, IC1.GND, R14.2, R17.2, R18.2, U3.VSS
- net HOLD: now also U2.PD0
- net LED: now also U2.PF4
- net N$2: now also C15.1, IC1.OUT, U3.VINA+; no longer R6.1, R8.2, U$3.VREF
- net N$3: now also R14.1, R15.2, R17.1, R18.1, T1.E; no longer R5.2, R7.2, U$3.VOUT
- net RESET: now also ISP.3; no longer ISP.2
- net S+: now also LSP2.MP; no longer X2.1
- net S-: now also LSP3.MP; no longer X3.1
- net SCK: now also ISP.6; no longer ISP.3
- net V+: now also D1.C, LSP1.MP; no longer X1.1
- net V-: now also LSP4.MP, T1.C; no longer X4.1
- net VCC: now also C18.2, ISP.2, S2.2; no longer ISP.6
- net VCCA: now also C14.1, C16.1, D1.A, IC1.VIN, U3.VDD; no longer U1.VIN
Other:
- moved on the sheet: D1, T1

Commit message: updated project
Parts:
- removed USART: (no value), con-lstb:MA03-1
- added SV1: (no value), con-lstb:MA04-1
Connections:
- removed net (TOSC1)_XTAL1: U2.(TOSC1)_XTAL1
- removed net (TOSC2)_XTAL2: U2.(TOSC2)_XTAL2
- net GND: now also SV1.1; no longer USART.1
- net RX: now also SV1.2; no longer USART.2
- net TX: now also SV1.3; no longer USART.3
- net VCC: now also SV1.4
Other:
- moved on the sheet: C15
