File: miliohmeter/main2.brd (EAGLE design)
At the start: 59.7 x 54.3 mm, 62 parts, among them IC1 LT1019S-2.5, IC2 7805TV, U2 ATMEGA169P-16AU, U3 MCP6V02-E/SN

Commit message: aeaz
Parts:
- renumbered IC2 to REG1, JP1 to PWR, JP2 to ISP, LSP1 to V+, LSP2 to S+, LSP3 to S-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
