File: mains_timer/main.sch (EAGLE design)
At the start: 0 parts

Commit message: a
Parts:
- added C1: 100u, rcl:C-US025-025X050
- added C2: 100n, rcl:C-US025-025X050
- added C3: 100u, rcl:CPOL-USE2-5
- added C4: 100n, rcl:CPOL-USE2-5
- added IC1: 4060N, 40xx:4060N
- added IC2: 7812TV, linear:7812TV
- added POWER, SW: (no value), pinhead:PINHD-1X2
- added U$1: 835-1A_RELAY12V, 7_segment_lib:835-1A_RELAY12V
Connections:
- new net 12V: C2.1, C3.+, IC2.VO, U$1.COIL1
- new net GND: C1.2, C2.2, C3.-, C4.-, IC2.GND, POWER.1
- new net VDD: C1.1, C4.+, IC2.VI, POWER.2
