File: mains_timer/main.sch (EAGLE design)
At the start: 9 parts, among them IC1 4060N, IC2 7812TV

Commit message: a
Parts:
- removed IC1: 4060N, 40xx:4060N
- added U$2: KBP205GK, 7_segment_lib:KBP205GK
Connections:
- new net N$1: POWER.2, U$2.AC@2
- new net N$2: POWER.1, U$2.AC@1
- net GND: now also U$2.-; no longer POWER.1
- net VDD: now also U$2.+; no longer POWER.2
Changed lines of the file:
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@@
 <parts>
 <part name="U$1" library="7_segment_lib" library_urn="urn:adsk.eagle:library:1964360" deviceset="835-1A_RELAY12V" device=""/>
-<part name="IC1" library="40xx" library_urn="urn:adsk.eagle:library:80" deviceset="4060" device="N" package3d_urn="urn:adsk.eagle:package:922/2"/>
 <part name="POWER" library="pinhead" library_urn="urn:adsk.eagle:library:325" deviceset="PINHD-1X2" device="" package3d_urn="urn:adsk.eagle:package:22435/2"/>
 <part name="SW" library="pinhead" library_urn="urn:adsk.eagle:library:325" deviceset="PINHD-1X2" device="" package3d_urn="urn:adsk.eagle:package:22435/2"/>
@@
 <part name="SUPPLY3" library="SparkFun-PowerSymbols" library_urn="urn:adsk.eagle:library:530" deviceset="VDD" device=""/>
 <part name="SUPPLY4" library="SparkFun-PowerSymbols" library_urn="urn:adsk.eagle:library:530" deviceset="12V" device=""/>
+<part name="U$2" library="7_segment_lib" library_urn="urn:adsk.eagle:library:1964360" deviceset="KBP205G" device="K" package3d_urn="urn:adsk.eagle:package:6702032/1"/>
 </parts>
 <sheets>
@@
 <attribute name="VALUE" x="-7.62" y="-9.652" size="1.778" layer="96" font="vector"/>
 </instance>
-<instance part="IC1" gate="A" x="0" y="-43.18" smashed="yes">
-<attribute name="NAME" x="-7.62" y="-24.765" size="1.778" layer="95"/>
-<attribute name="VALUE" x="-7.62" y="-63.5" size="1.778" layer="96"/>
-</instance>
 <instance part="POWER" gate="G$1" x="-91.44" y="-40.64" smashed="yes" rot="R180">
 <attribute name="NAME" x="-85.09" y="-46.355" size="1.778" layer="95" rot="R180"/>
@@
 <attribute name="VALUE" x="-62.23" y="-33.02" size="1.778" layer="96"/>
 </instance>
-<instance part="GND1" gate="1" x="-81.28" y="-45.72" smashed="yes">
-<attribute name="VALUE" x="-81.28" y="-45.974" size="1.778" layer="96" align="top-center"/>
+<instance part="GND1" gate="1" x="-71.12" y="-48.26" smashed="yes">
+<attribute name="VALUE" x="-71.12" y="-48.514" size="1.778" layer="96" align="top-center"/>
 </instance>
 <instance part="SUPPLY1" gate="G$1" x="-10.16" y="5.08" smashed="yes">
 <attribute name="VALUE" x="-10.16" y="7.874" size="1.778" layer="96" align="bottom-center"/>
 </instance>
-<instance part="SUPPLY2" gate="VDD" x="-81.28" y="-40.64" smashed="yes">
-<attribute name="VALUE" x="-81.28" y="-37.846" size="1.778" layer="96" align="bottom-center"/>
+<instance part="SUPPLY2" gate="VDD" x="-71.12" y="-30.48" smashed="yes">
+<attribute name="VALUE" x="-71.12" y="-27.686" size="1.778" layer="96" align="bottom-center"/>
 </instance>
 <instance part="IC2" gate="A1" x="-55.88" y="-60.96" smashed="yes">
@@
 <attribute name="VALUE" x="-40.64" y="-55.626" size="1.778" layer="96" align="bottom-center"/>
 </instance>
+<instance part="U$2" gate="G$1" x="-71.12" y="-40.64" smashed="yes" rot="R270">
+<attribute name="NAME" x="-66.929" y="-34.036" size="1.778" layer="95" rot="R270"/>
+<attribute name="VALUE" x="-76.835" y="-34.036" size="1.778" layer="96" rot="R270"/>
+</instance>
 </instances>
 <busses>
@@
 <nets>
 <net name="VDD" class="0">
-<segment>
-<pinref part="POWER" gate="G$1" pin="2"/>
-<pinref part="SUPPLY2" gate="VDD" pin="VDD"/>
-<wire x1="-81.28" y1="-40.64" x2="-88.9" y2="-40.64" width="0.1524" layer="91"/>
-</segment>
 <segment>
 <pinref part="C1" gate="G$1" pin="1"/>
@@
 <wire x1="-73.66" y1="-60.96" x2="-73.66" y2="-58.42" width="0.1524" layer="91"/>
 </segment>
+<segment>
+<pinref part="U$2" gate="G$1" pin="+"/>
+<pinref part="SUPPLY2" gate="VDD" pin="VDD"/>
+</segment>
 </net>
 <net name="GND" class="0">
-<segment>
-<pinref part="POWER" gate="G$1" pin="1"/>
-<pinref part="GND1" gate="1" pin="GND"/>
-<wire x1="-81.28" y1="-43.18" x2="-88.9" y2="-43.18" width="0.1524" layer="91"/>
-</segment>
 <segment>
 <pinref part="C1" gate="G$1" pin="2"/>
@@
 <pinref part="GND2" gate="1" pin="GND"/>
 </segment>
+<segment>
+<pinref part="U$2" gate="G$1" pin="-"/>
+<pinref part="GND1" gate="1" pin="GND"/>
+</segment>
 </net>
 <net name="12V" class="0">
@@
 </segment>
 </net>
+<net name="N$1" class="0">
+<segment>
+<pinref part="U$2" gate="G$1" pin="AC@2"/>
+<wire x1="-73.66" y1="-38.1" x2="-81.28" y2="-38.1" width="0.1524" layer="91"/>
+<wire x1="-81.28" y1="-38.1" x2="-81.28" y2="-40.64" width="0.1524" layer="91"/>
+<pinref part="POWER" gate="G$1" pin="2"/>
+<wire x1="-81.28" y1="-40.64" x2="-88.9" y2="-40.64" width="0.1524" layer="91"/>
+</segment>
+</net>
+<net name="N$2" class="0">
+<segment>
+<pinref part="POWER" gate="G$1" pin="1"/>
+<wire x1="-88.9" y1="-43.18" x2="-81.28" y2="-43.18" width="0.1524" layer="91"/>
+<wire x1="-81.28" y1="-43.18" x2="-81.28" y2="-45.72" width="0.1524" layer="91"/>
+<wire x1="-81.28" y1="-45.72" x2="-66.04" y2="-45.72" width="0.1524" layer="91"/>
+<wire x1="-66.04" y1="-45.72" x2="-66.04" y2="-38.1" width="0.1524" layer="91"/>
+<pinref part="U$2" gate="G$1" pin="AC@1"/>
+<wire x1="-66.04" y1="-38.1" x2="-68.58" y2="-38.1" width="0.1524" layer="91"/>
+</segment>
+</net>
