File: mains_timer/main1.sch (EAGLE design)
At the start: 25 parts, among them IC1 4060N, IC2 7812TV, IC3 4060N, IC4 4017N, T1 2N2222, Y1 32.768kHz

Commit message: a
Parts:
- removed POWER: (no value), pinhead:PINHD-1X2
- added PAD1, PAD2: (no value), 7_segment_lib:2,54/1,0
- C1: value 100u -> 100n
- LED1: device led:LED5MM -> led:LED3MM
- R4: device rcl:R-US_0207/7 -> rcl:R-US_0207/2V
Connections:
- new net N$24: PAD2.P, U$3.MAIN
- net N$1: no longer POWER.2
- net N$2: no longer POWER.1
- net N$23: now also PAD1.P, U$3.NO; no longer IC3A.Q4, LED1.A
- net N$6: now also LED1.A
Other:
- moved on the sheet: LED1, R5
Changed lines of the file:
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@@
 </classes>
 <parts>
-<part name="POWER" library="pinhead" library_urn="urn:adsk.eagle:library:325" deviceset="PINHD-1X2" device="" package3d_urn="urn:adsk.eagle:package:22435/2"/>
 <part name="SW" library="pinhead" library_urn="urn:adsk.eagle:library:325" deviceset="PINHD-1X2" device="" package3d_urn="urn:adsk.eagle:package:22435/2"/>
 <part name="GND1" library="SparkFun-PowerSymbols" library_urn="urn:adsk.eagle:library:530" deviceset="GND" device=""/>
 <part name="SUPPLY2" library="SparkFun-PowerSymbols" library_urn="urn:adsk.eagle:library:530" deviceset="VDD" device=""/>
 <part name="IC2" library="linear" library_urn="urn:adsk.eagle:library:262" deviceset="78*" device="TV" package3d_urn="urn:adsk.eagle:package:16417/1" technology="12"/>
-<part name="C1" library="rcl" library_urn="urn:adsk.eagle:library:334" deviceset="C-US" device="025-025X050" package3d_urn="urn:adsk.eagle:package:23629/2" value="100u"/>
+<part name="C1" library="rcl" library_urn="urn:adsk.eagle:library:334" deviceset="C-US" device="025-025X050" package3d_urn="urn:adsk.eagle:package:23629/2" value="100n"/>
 <part name="C2" library="rcl" library_urn="urn:adsk.eagle:library:334" deviceset="C-US" device="025-025X050" package3d_urn="urn:adsk.eagle:package:23629/2" value="100n"/>
 <part name="C3" library="rcl" library_urn="urn:adsk.eagle:library:334" deviceset="CPOL-US" device="E2-5" package3d_urn="urn:adsk.eagle:package:23346/2" value="100u"/>
@@
 <part name="T1" library="adafruit" library_urn="urn:adsk.eagle:library:420" deviceset="2N2222" device="" package3d_urn="urn:adsk.eagle:package:6240647/1"/>
 <part name="GND5" library="SparkFun-PowerSymbols" library_urn="urn:adsk.eagle:library:530" deviceset="GND" device=""/>
-<part name="R4" library="rcl" library_urn="urn:adsk.eagle:library:334" deviceset="R-US_" device="0207/7" package3d_urn="urn:adsk.eagle:package:23493/1"/>
+<part name="R4" library="rcl" library_urn="urn:adsk.eagle:library:334" deviceset="R-US_" device="0207/2V" package3d_urn="urn:adsk.eagle:package:23490/1"/>
 <part name="U$3" library="7_segment_lib" library_urn="urn:adsk.eagle:library:1964360" deviceset="835-1A_RELAY12V" device=""/>
 <part name="SUPPLY6" library="SparkFun-PowerSymbols" library_urn="urn:adsk.eagle:library:530" deviceset="12V" device=""/>
 <part name="GND6" library="SparkFun-PowerSymbols" library_urn="urn:adsk.eagle:library:530" deviceset="GND" device=""/>
-<part name="LED1" library="led" library_urn="urn:adsk.eagle:library:259" deviceset="LED" device="5MM" package3d_urn="urn:adsk.eagle:package:15799/2"/>
+<part name="LED1" library="led" library_urn="urn:adsk.eagle:library:259" deviceset="LED" device="3MM" package3d_urn="urn:adsk.eagle:package:15797/1"/>
 <part name="R5" library="rcl" library_urn="urn:adsk.eagle:library:334" deviceset="R-US_" device="0207/7" package3d_urn="urn:adsk.eagle:package:23493/1" value="500"/>
 <part name="GND7" library="SparkFun-PowerSymbols" library_urn="urn:adsk.eagle:library:530" deviceset="GND" device=""/>
+<part name="PAD1" library="7_segment_lib" library_urn="urn:adsk.eagle:library:1964360" deviceset="2,54/1,0" device="" package3d_urn="urn:adsk.eagle:package:1964566/3"/>
+<part name="PAD2" library="7_segment_lib" library_urn="urn:adsk.eagle:library:1964360" deviceset="2,54/1,0" device="" package3d_urn="urn:adsk.eagle:package:1964566/3"/>
 </parts>
 <sheets>
@@
 </plain>
 <instances>
-<instance part="POWER" gate="G$1" x="-137.16" y="-66.04" smashed="yes" rot="R180">
-<attribute name="NAME" x="-130.81" y="-71.755" size="1.778" layer="95" rot="R180"/>
-<attribute name="VALUE" x="-130.81" y="-60.96" size="1.778" layer="96" rot="R180"/>
-</instance>
 <instance part="SW" gate="G$1" x="7.62" y="-45.72" smashed="yes" rot="R180">
 <attribute name="NAME" x="13.97" y="-51.435" size="1.778" layer="95" rot="R180"/>
@@
 <attribute name="VALUE" x="137.16" y="-73.914" size="1.778" layer="96" align="top-center"/>
 </instance>
-<instance part="LED1" gate="G$1" x="121.92" y="-40.64" smashed="yes" rot="R90">
-<attribute name="NAME" x="126.492" y="-37.084" size="1.778" layer="95" rot="R180"/>
-<attribute name="VALUE" x="126.492" y="-34.925" size="1.778" layer="96" rot="R180"/>
-</instance>
-<instance part="R5" gate="G$1" x="129.54" y="-45.72" smashed="yes" rot="R90">
-<attribute name="NAME" x="128.0414" y="-49.53" size="1.778" layer="95" rot="R90"/>
-<attribute name="VALUE" x="132.842" y="-49.53" size="1.778" layer="96" rot="R90"/>
-</instance>
-<instance part="GND7" gate="1" x="129.54" y="-53.34" smashed="yes">
-<attribute name="VALUE" x="129.54" y="-53.594" size="1.778" layer="96" align="top-center"/>
+<instance part="LED1" gate="G$1" x="91.44" y="-43.18" smashed="yes">
+<attribute name="NAME" x="94.996" y="-47.752" size="1.778" layer="95" rot="R90"/>
+<attribute name="VALUE" x="97.155" y="-47.752" size="1.778" layer="96" rot="R90"/>
+</instance>
+<instance part="R5" gate="G$1" x="91.44" y="-53.34" smashed="yes" rot="R90">
+<attribute name="NAME" x="89.9414" y="-57.15" size="1.778" layer="95" rot="R90"/>
+<attribute name="VALUE" x="94.742" y="-57.15" size="1.778" layer="96" rot="R90"/>
+</instance>
+<instance part="GND7" gate="1" x="91.44" y="-60.96" smashed="yes">
+<attribute name="VALUE" x="91.44" y="-61.214" size="1.778" layer="96" align="top-center"/>
+</instance>
+<instance part="PAD1" gate="P" x="218.44" y="-63.5" smashed="yes" rot="R90">
+<attribute name="NAME" x="216.5858" y="-64.643" size="1.778" layer="95" rot="R90"/>
+<attribute name="VALUE" x="221.742" y="-64.643" size="1.778" layer="96" rot="R90"/>
+</instance>
+<instance part="PAD2" gate="P" x="218.44" y="-38.1" smashed="yes" rot="R270">
+<attribute name="NAME" x="220.2942" y="-36.957" size="1.778" layer="95" rot="R270"/>
+<attribute name="VALUE" x="215.138" y="-36.957" size="1.778" layer="96" rot="R270"/>
 </instance>
 </instances>
@@
 <wire x1="-119.38" y1="-60.96" x2="-127" y2="-60.96" width="0.1524" layer="91"/>
 <wire x1="-127" y1="-60.96" x2="-127" y2="-66.04" width="0.1524" layer="91"/>
-<pinref part="POWER" gate="G$1" pin="2"/>
 <wire x1="-127" y1="-66.04" x2="-134.62" y2="-66.04" width="0.1524" layer="91"/>
 </segment>
@@
 <net name="N$2" class="0">
 <segment>
-<pinref part="POWER" gate="G$1" pin="1"/>
 <wire x1="-134.62" y1="-68.58" x2="-127" y2="-68.58" width="0.1524" layer="91"/>
 <wire x1="-127" y1="-68.58" x2="-127" y2="-73.66" width="0.1524" layer="91"/>
@@
 <segment>
 <pinref part="IC1" gate="A" pin="Q14"/>
-<wire x1="50.8" y1="-40.64" x2="93.98" y2="-40.64" width="0.1524" layer="91"/>
+<wire x1="50.8" y1="-40.64" x2="91.44" y2="-40.64" width="0.1524" layer="91"/>
 <pinref part="IC3" gate="A" pin="P1"/>
+<pinref part="LED1" gate="G$1" pin="A"/>
+<wire x1="91.44" y1="-40.64" x2="93.98" y2="-40.64" width="0.1524" layer="91"/>
+<junction x="91.44" y="-40.64"/>
 </segment>
 </net>
@@
 <pinref part="LED1" gate="G$1" pin="C"/>
 <pinref part="R5" gate="G$1" pin="2"/>
-<wire x1="127" y1="-40.64" x2="129.54" y2="-40.64" width="0.1524" layer="91"/>
 </segment>
 </net>
 <net name="N$23" class="0">
 <segment>
-<pinref part="IC3" gate="A" pin="Q4"/>
-<pinref part="LED1" gate="G$1" pin="A"/>
-</segment>
-</net>
+<pinref part="U$3" gate="G$1" pin="NO"/>
+<pinref part="PAD1" gate="P" pin="P"/>
+</segment>
+</net>
+<net name="N$24" class="0">
+<segment>
+<pinref part="U$3" gate="G$1" pin="MAIN"/>
+<pinref part="PAD2" gate="P" pin="P"/>
+</segment>
+</net>
