File: HV9925/main.brd (EAGLE design)
At the start: 160 x 100 mm, 23 parts

Commit message: update
Parts:
- added J1: USBSMD, SparkFun-Retired:USB-MINIB
Changed lines of the file:
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@@
 <?xml version="1.0" encoding="utf-8"?>
 <!DOCTYPE eagle SYSTEM "eagle.dtd">
-<eagle version="8.7.1">
+<eagle version="9.0.1">
 <drawing>
 <settings>
@@
 <setting verticaltext="up"/>
 </settings>
-<grid distance="12.7" unitdist="mil" unit="mil" style="dots" multiple="1" display="yes" altdistance="5" altunitdist="mil" altunit="mil"/>
+<grid distance="0.003125" unitdist="mic" unit="mm" style="dots" multiple="1" display="yes" altdistance="5" altunitdist="mil" altunit="mil"/>
 <layers>
 <layer number="1" name="Top" color="4" fill="1" visible="yes" active="yes"/>
@@
 <element name="U$8" library="7_segment_lib" library_urn="urn:adsk.eagle:library:1964360" package="PLCC2_3528" value="PLCC2_3528" x="-35.56" y="35.56"/>
 <element name="U$9" library="7_segment_lib" library_urn="urn:adsk.eagle:library:1964360" package="PLCC2_3528" value="PLCC2_3528" x="-40.64" y="35.56"/>
+<element name="J1" library="SparkFun-Retired" library_urn="urn:adsk.eagle:library:533" package="USB-MINIB" value="USBSMD" x="32.90315625" y="76.451459375">
+<attribute name="PROD_ID" value="CONN-08193" x="32.90315625" y="76.451459375" size="1.778" layer="27" display="off"/>
+</element>
 </elements>
 <signals>
