File: HV9925/main.sch (EAGLE design)
At the start: 23 parts

Commit message: update
Parts:
- added J1: USBSMD, SparkFun-Retired:USBSMD
Changed lines of the file:
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@@
 <?xml version="1.0" encoding="utf-8"?>
 <!DOCTYPE eagle SYSTEM "eagle.dtd">
-<eagle version="8.7.1">
+<eagle version="9.0.1">
 <drawing>
 <settings>
@@
 <part name="C3" library="rcl" library_urn="urn:adsk.eagle:library:334" deviceset="C-US" device="025-025X050" package3d_urn="urn:adsk.eagle:package:23629/2" value="10n"/>
 <part name="R2" library="rcl" library_urn="urn:adsk.eagle:library:334" deviceset="R-US_" device="R0805" package3d_urn="urn:adsk.eagle:package:23553/2" value="20"/>
+<part name="J1" library="SparkFun-Retired" library_urn="urn:adsk.eagle:library:533" deviceset="USB" device="SMD"/>
 </parts>
 <sheets>
@@
 <instance part="C3" gate="G$1" x="17.78" y="-27.94"/>
 <instance part="R2" gate="G$1" x="-5.08" y="-30.48" rot="R90"/>
+<instance part="J1" gate="G$1" x="-96.52" y="-12.7"/>
 </instances>
 <busses>
