File: ATmega406/main.sch (EAGLE design)
At the start: 9 parts, among them Q1 16M

Commit message: afb
Parts:
- added C4, C5: 10u, rcl:C-USC0805
- added J2: (no value), Wurth_Elektronik_Electromechanic_Terminal_Blocks_Connectors_rev17a:691136710007
- added R5, R6, R7, R8, RSC: (no value), rcl:R-US_R0805
- added RSC+, RSC-: (no value), 7_segment_lib:2,54/1,0
- added SV1: (no value), con-lstb:MA03-1
Connections:
- net N$9 renamed VCC
- new net BAT+: J2.6, R3.2
- new net BAT-: J2.2, R2.2, R8.2, RSC+.P, RSC.1
- new net BAT1: J2.3, R7.2
- new net BAT2: J2.4, R6.2
- new net BAT3: J2.5, R5.2
- new net GND: C2.2, C3.2, C4.2, C5.2, J2.1, R1.2, RSC-.P, RSC.2, SV1.3, U$1.GND@1, U$1.GND@2, U$1.GND@3, U$1.GND@4, U$1.SGND, U$1.VREFGND
- new net N$10: R6.1, U$1.PV2
- new net N$11: R7.1, U$1.PV1
- new net N$12: R8.1, U$1.NV
- new net N$9: C5.1, U$1.VREF
- new net SCL: SV1.1, U$1.SCL
- new net SDA: SV1.2, U$1.SDA
- new net VIN: J2.7, U$1.VFET
- net N$1: now also C4.1, U$1.VREG; no longer C2.2, C3.2, U$1.GND@1, U$1.GND@2, U$1.GND@3, U$1.GND@4, U$1.SGND, U$1.VREFGND
- net N$2: now also C1.1
- net N$3: now also U$1.PV4; no longer C1.2, R2.2
- net N$4: now also R5.1, U$1.PV3; no longer C1.1, R1.2, R3.2
- net N$5: now also C1.2
Other:
- moved on the sheet: C1, R1, R2, R3, R4
