File: MCP2210/main.brd (EAGLE design)
At the start: 26 x 18.7 mm, 11 parts, among them J1 USB_A_SMT_MALE, Q1 12MHz

Commit message: started new layout
Parts:
- removed R2, R3: 470, resistor:R0603
- removed U$2: BICOLOR_LED, 7_segment_lib:BICOLOR_LED
Connections:
- removed net N$10: R3.2, U$2.C1
- removed net N$11: R3.1, U$1.6
- removed net N$12: R2.1, U$1.8
- removed net N$3: C1.2, C2.2, C3.2, C4.2, J1.GND1, J1.SHLD1, J1.SHLD2, SV1.3, U$1.20
- removed net N$9: R2.2, U$2.C2
- new net GND: C1.2, C2.2, C3.2, C4.2, J1.GND1, J1.SHLD1, J1.SHLD2, SV1.5, U$1.20
- net N$4: now also SV1.3; no longer SV1.5, U$2.A1, U$2.A2
Routing:
- net GND: track 0.00 -> 33.1 mm
- net N$3: track 17.5 -> 0.00 mm
- net N$4: track 5.78 -> 21.6 mm
- net N$7: track 0.00 -> 9.58 mm
- net N$15: track 0.00 -> 5.47 mm
- added copper zone on layer 1, net GND
Other:
- board size 26 x 18.7 mm -> 25.5 x 18.1 mm
