File: MCP2210/main.sch (EAGLE design)
At the start: 11 parts, among them J1 USB_A_SMT_MALE, Q1 12MHz

Commit message: started new layout
Parts:
- removed R2, R3: 470, resistor:R-US_R0603
- removed U$2: BICOLOR_LED, 7_segment_lib:BICOLOR_LED
Connections:
- removed net N$10: R3.2, U$2.C1
- removed net N$11: R3.1, U$1.GP1
- removed net N$12: R2.1, U$1.GP3
- removed net N$3: C1.2, C2.2, C3.2, C4.2, J1.GND, J1.SHIELD, SV1.3, U$1.VSS
- removed net N$9: R2.2, U$2.C2
- new net GND: C1.2, C2.2, C3.2, C4.2, J1.GND, J1.SHIELD, SV1.5, U$1.VSS
- net N$4: now also SV1.3; no longer SV1.5, U$2.A1, U$2.A2
