File: MCP2210/main1.sch (EAGLE design)
At the start: 11 parts, among them J1 USB_A_SMT_MALE, Q1 12MHz

Commit message: added 2nd layout
Parts:
- added R1: 10k, resistor:R-US_R0603
Connections:
- new net N$8: R1.1, U$1.RESET
- net N$3: now also SV1.5; no longer SV1.3
- net N$4: now also R1.2, SV1.3; no longer SV1.5
Changed lines of the file:
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@@
 <part name="R3" library="resistor" library_urn="urn:adsk.eagle:library:348" deviceset="R-US_" device="R0603" package3d_urn="urn:adsk.eagle:package:23555/2" value="470"/>
 <part name="SV1" library="con-lstb" library_urn="urn:adsk.eagle:library:162" deviceset="MA05-1" device="" package3d_urn="urn:adsk.eagle:package:8332/1"/>
+<part name="R1" library="resistor" library_urn="urn:adsk.eagle:library:348" deviceset="R-US_" device="R0603" package3d_urn="urn:adsk.eagle:package:23555/2" value="10k"/>
 </parts>
 <sheets>
@@
 <attribute name="VALUE" x="1.27" y="17.78" size="1.778" layer="96"/>
 <attribute name="NAME" x="1.27" y="36.322" size="1.778" layer="95"/>
+</instance>
+<instance part="R1" gate="G$1" x="45.72" y="55.88" rot="R90">
+<attribute name="NAME" x="44.2214" y="52.07" size="1.778" layer="95" rot="R90"/>
+<attribute name="VALUE" x="49.022" y="52.07" size="1.778" layer="96" rot="R90"/>
 </instance>
 </instances>
@@
 <wire x1="25.4" y1="48.26" x2="35.56" y2="48.26" width="0.1524" layer="91"/>
 <junction x="25.4" y="48.26"/>
-<pinref part="SV1" gate="G$1" pin="3"/>
-<wire x1="10.16" y1="27.94" x2="22.86" y2="12.7" width="0.1524" layer="91"/>
+<pinref part="SV1" gate="G$1" pin="5"/>
+<wire x1="10.16" y1="33.02" x2="22.86" y2="12.7" width="0.1524" layer="91"/>
 <junction x="22.86" y="12.7"/>
 <wire x1="15.24" y1="48.26" x2="15.24" y2="53.34" width="0.1524" layer="91"/>
@@
 <wire x1="20.32" y1="40.64" x2="20.32" y2="22.86" width="0.1524" layer="91"/>
 <junction x="20.32" y="40.64"/>
-<pinref part="SV1" gate="G$1" pin="5"/>
-<wire x1="20.32" y1="22.86" x2="10.16" y2="33.02" width="0.1524" layer="91"/>
+<pinref part="SV1" gate="G$1" pin="3"/>
+<wire x1="20.32" y1="22.86" x2="10.16" y2="27.94" width="0.1524" layer="91"/>
+<pinref part="R1" gate="G$1" pin="2"/>
+<wire x1="45.72" y1="60.96" x2="45.72" y2="71.12" width="0.1524" layer="91"/>
+<junction x="45.72" y="71.12"/>
 </segment>
 </net>
@@
 </segment>
 </net>
+<net name="N$8" class="0">
+<segment>
+<pinref part="U$1" gate="G$1" pin="RESET"/>
+<pinref part="R1" gate="G$1" pin="1"/>
+</segment>
+</net>

Commit message: started new layout
Parts:
- Q1: device crystal:CRYSTALHC49U-V -> crystal:CRYSTALSM49
Connections:
- net N$1 renamed N+
- net N$2 renamed N-
Changed lines of the file:
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@@
 <parts>
 <part name="J1" library="SparkFun-Connectors" library_urn="urn:adsk.eagle:library:513" deviceset="USB_A" device="_SMT_MALE" package3d_urn="urn:adsk.eagle:package:38305/1"/>
-<part name="Q1" library="crystal" library_urn="urn:adsk.eagle:library:204" deviceset="CRYSTAL" device="HC49U-V" package3d_urn="urn:adsk.eagle:package:12075/1" value="12MHz"/>
+<part name="Q1" library="crystal" library_urn="urn:adsk.eagle:library:204" deviceset="CRYSTAL" device="SM49" package3d_urn="urn:adsk.eagle:package:12085/1" value="12MHz"/>
 <part name="U$1" library="7_segment_lib" library_urn="urn:adsk.eagle:library:1964360" deviceset="MCP2210" device="" package3d_urn="urn:adsk.eagle:package:7942598/1"/>
 <part name="C1" library="rcl" library_urn="urn:adsk.eagle:library:334" deviceset="C-US" device="C0805" package3d_urn="urn:adsk.eagle:package:23617/2" value="100n"/>
@@
 </busses>
 <nets>
-<net name="N$1" class="0">
+<net name="N+" class="0">
 <segment>
 <pinref part="J1" gate="G$1" pin="D+"/>
 <pinref part="U$1" gate="G$1" pin="D+"/>
 <wire x1="15.24" y1="45.72" x2="45.72" y2="45.72" width="0.1524" layer="91"/>
+<label x="17.78" y="45.72" size="1.778" layer="95"/>
 </segment>
 </net>
-<net name="N$2" class="0">
+<net name="N-" class="0">
 <segment>
 <pinref part="U$1" gate="G$1" pin="D-"/>
 <pinref part="J1" gate="G$1" pin="D-"/>
 <wire x1="45.72" y1="43.18" x2="15.24" y2="43.18" width="0.1524" layer="91"/>
+<label x="17.78" y="43.18" size="1.778" layer="95"/>
 </segment>
 </net>

Commit message: -ma
Connections:
- net N+ renamed N_P
- net N- renamed N_N
Changed lines of the file:
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@@
 </busses>
 <nets>
-<net name="N+" class="0">
+<net name="N_P" class="0">
 <segment>
 <pinref part="J1" gate="G$1" pin="D+"/>
@@
 </segment>
 </net>
-<net name="N-" class="0">
+<net name="N_N" class="0">
 <segment>
 <pinref part="U$1" gate="G$1" pin="D-"/>
