File: WaveP/main.brd (EAGLE design)
At the start: 57 x 45 mm, 41 parts, among them Q1 16MHz, U1 328P, X1 MINI-USB_SHIELD5P2-32005-601, X2 1503_09

Commit message: -a
a
Parts:
- added U$4: PC_SPDT_SWITCH, 7_segment_lib:PC_SPDT_SWITCH
- added U2: MCP6291T, 7_segment_lib:SOT23-5
- moved OUT 50.1 mm to (16.7, 33.3), turned to 90 degrees
- moved C10 48.4 mm to (22.1, 35.7)
- moved C4 48.4 mm to (22.1, 41.9)
- moved C5 48.4 mm to (26.0, 41.4)
- moved POT 48.4 mm to (16.6, 40.0)
- moved R6 48.4 mm to (19.6, 41.9)
- moved R7 48.4 mm to (24.7, 35.7)
- moved U$2 48.4 mm to (23.4, 35.1)
Connections:
- removed net OUT: OUT.1, POT.2
- new net N$11: POT.2, U2.3
- new net N$2: OUT.1, U2.1, U2.4
- new net VCC: C1.1, C10.1, C11.1, C12.1, ISP.6, R10.2, R7.1, R8.1, R9.2, SV1.5, SV1.5@1, SV2.VCC, U$2.1, U$4.NO, U1.20, U1.21, U1.7, U2.2
- net GND: now also U2.5, X2.1
- net V_BATT: now also U$4.COM; no longer C1.1, C10.1, C11.1, C12.1, ISP.6, R10.2, R7.1, R8.1, R9.2, SV1.5, SV1.5@1, SV2.VCC, U$2.1, U1.20, U1.21, U1.7

Commit message: -a
a
Parts:
- added C13: 100u, rcl:E2-5
Connections:
- new net N$10: C13.-, OUT.1, X2.2, X2.3
- net N$2: now also C13.+; no longer OUT.1
Changed lines of the file:
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@@
 <attribute name="NAME" x="-7" y="-8" size="1.27" layer="21" align="center"/>
+</element>
+<element name="C13" library="rcl" library_urn="urn:adsk.eagle:library:334" package="E2-5" package3d_urn="urn:adsk.eagle:package:23346/2" value="100u" x="-8.5" y="-13.5" smashed="yes">
+<attribute name="NAME" x="-5.96" y="-12.484" size="1.27" layer="25" ratio="10"/>
+<attribute name="SPICEPREFIX" value="C" x="-8.5" y="-13.5" size="1.778" layer="27" display="off"/>
+<attribute name="VALUE" x="-5.96" y="-15.659" size="1.27" layer="27" ratio="10"/>
 </element>
 </elements>
@@
 <contactref element="U2" pad="4"/>
 <contactref element="U2" pad="1"/>
-<contactref element="OUT" pad="1"/>
-<wire x1="-9.05" y1="1.3001" x2="16.74" y2="31.99875" width="0" layer="19" extent="1-1"/>
-<wire x1="-10.95" y1="-1.3001" x2="-9.05" y2="1.3001" width="0" layer="19" extent="1-1"/>
+<contactref element="C13" pad="+"/>
+<wire x1="-10.95" y1="-1.3001" x2="-9.516" y2="-13.5" width="0" layer="19" extent="1-1"/>
+<wire x1="-9.05" y1="1.3001" x2="-10.95" y2="-1.3001" width="0" layer="19" extent="1-1"/>
 </signal>
 <signal name="N$11">
@@
 <wire x1="-9.05" y1="-1.3001" x2="16.59375" y2="40.00125" width="0" layer="19" extent="1-1"/>
 </signal>
+<signal name="N$10">
+<contactref element="X2" pad="3"/>
+<contactref element="X2" pad="2"/>
+<contactref element="C13" pad="-"/>
+<contactref element="OUT" pad="1"/>
+<wire x1="6.19" y1="32.1" x2="10.69" y2="41.7" width="0" layer="19" extent="1-1"/>
+<wire x1="16.74" y1="31.99875" x2="6.19" y2="32.1" width="0" layer="19" extent="1-1"/>
+<wire x1="-7.484" y1="-13.5" x2="6.19" y2="32.1" width="0" layer="19" extent="1-1"/>
+</signal>
 </signals>

Commit message: -a
a
Parts:
- removed POT: 10k, con-lstb:MA03-1
- added TM1: (no value), adafruit:TRIM-3386
- C13: device rcl:E2-5 -> rcl:E2,5-6E
- moved C13 72.7 mm to (39.0, 41.5), flipped to the bottom, turned to 180 degrees
- moved U2 57.8 mm to (36.0, 35.0), flipped to the bottom, turned to 90 degrees
- moved X2 55.4 mm to (56.2, 38.4), turned to 270 degrees
- moved OUT 23.6 mm to (40.3, 35.7), turned to 270 degrees
- moved U$4 23.1 mm to (7.14, 14.2), turned to 270 degrees
- moved C1 18.1 mm to (28.3, 21.3), turned to 180 degrees
- moved C2 17.7 mm to (15.7, 8.79), turned to 0 degrees
- moved C12 17.1 mm to (48.6, 14.9), turned to 270 degrees
- moved C5 7.21 mm to (22.0, 35.4)
- moved UART 6.10 mm to (16.7, 16.6)
- moved C10 5.59 mm to (16.6, 34.7)
- moved C4 5.59 mm to (16.6, 40.9)
- moved R6 5.59 mm to (14.1, 40.9)
- moved R7 5.59 mm to (19.2, 34.7)
- moved U$2 5.59 mm to (17.9, 34.1)
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Connections:
- net BTN_NEXT: now also U1.13; no longer U1.12
- net BTN_OK: now also U1.12; no longer U1.13
- net FILTEROUT: now also TM1.3; no longer POT.3
- net GND: now also TM1.1; no longer POT.1
- net N$11: now also TM1.2; no longer POT.2
- net VCC: now also U$4.COM; no longer U$4.NO
- net V_BATT: now also U$4.NO; no longer U$4.COM
Routing:
- net GND: track 0.00 -> 76.4 mm
- net VCC: track 0.00 -> 41.7 mm
- net V_USB: track 0.00 -> 32.4 mm
- net V_BATT: track 0.00 -> 22.8 mm
- net N$10: track 0.00 -> 21.8 mm
- net FILTEROUT: track 0.00 -> 19.5 mm
- net N$2: track 0.00 -> 9.78 mm
- net N$11: track 0.00 -> 8.73 mm
- net PB7(XTAL2/TOSC2): track 0.00 -> 6.20 mm
- net VREF: track 0.00 -> 4.30 mm
- net PB6(XTAL1/TOSC1): track 0.00 -> 3.81 mm
- net BTN_OK: track 0.00 -> 3.74 mm
- net BTN_NEXT: track 0.00 -> 3.74 mm
- net SCK: track 0.00 -> 3.18 mm
- net MOSI: track 0.00 -> 3.18 mm
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
Commit message: -a
a
Parts:
- moved R10 17.9 mm to (41.9, 22.0), turned to 90 degrees
- moved R9 17.9 mm to (39.5, 22.0), turned to 90 degrees
- moved C8 8.30 mm to (30.6, 12.3), turned to 0 degrees
- moved C9 6.85 mm to (45.7, 14.0), turned to 180 degrees
- moved R12 6.60 mm to (34.8, 11.3), turned to 90 degrees
- moved R11 6.36 mm to (43.8, 11.3), turned to 270 degrees
- moved S2 1.58 mm to (48.3, 7.11), turned to 270 degrees
- moved S1 0.15 mm to (30.5, 7.11), turned to 270 degrees
Connections:
- net LED: now also U1.5; no longer U1.14
- net LED1: now also U1.6; no longer U1.15
Routing:
- net GND: track 76.4 -> 105.9 mm
- net VCC: track 41.7 -> 66.5 mm
- net BTN_OK: track 3.74 -> 14.5 mm
- net BTN_NEXT: track 3.74 -> 10.9 mm
- net LED1: track 1.96 -> 0.69 mm
- net LED: track 1.76 -> 0.59 mm

Commit message: -a
a
Parts:
- removed U$1, U$3: BICOLOR_LED, 7_segment_lib:BICOLOR_LED
- added LED1, LED2, LED3, LED4: (no value), adafruit:LED3MM
- moved R1 26.5 mm to (20.8, 13.1), turned to 180 degrees
- moved R2 25.3 mm to (23.3, 14.4)
- moved R10 7.10 mm to (45.7, 16.0), turned to 180 degrees
- moved R3 5.22 mm to (22.9, 7.25), turned to 0 degrees
- moved U2 1.45 mm to (35.6, 36.4)
- moved UART 1.23 mm to (15.5, 16.8)
- moved ISP 0.89 mm to (35.7, 31.1)
- moved R4 0.72 mm to (22.4, 4.74)
- moved TM1 0.61 mm to (29.1, 38.3), turned to 90 degrees
Connections:
- net CS: now also U1.14; no longer U1.16
- net GND: now also R1.2, R2.2, U2.2; no longer U$1.C1, U$1.C2, U2.5
- net LED: now also LED1.A; no longer R1.1
- net LED1: now also LED2.A; no longer R2.1
- net N$3: now also LED3.K, R4.1; no longer R3.2, U$3.A2
- net N$4: now also LED4.K, R3.1; no longer R4.2, U$3.A1
- net N$6: now also R4.2; no longer U$3.C2
- net N$7: now also R3.2; no longer U$3.C1
- net N$8: now also LED2.K, R2.1; no longer R1.2, U$1.A1
- net N$9: now also LED1.K, R1.1; no longer R2.2, U$1.A2
- net VCC: now also U2.5; no longer U2.2
- net V_USB: now also LED3.A, LED4.A; no longer R3.1, R4.1
Routing:
- net VCC: track 66.5 -> 98.8 mm
- net GND: track 105.9 -> 137.1 mm
- net SCK: track 3.18 -> 21.4 mm
- net MISO: track 3.18 -> 18.8 mm
- net SDA: track 0.00 -> 6.56 mm
- net CS: track 0.00 -> 6.33 mm
- net N$11: track 8.73 -> 2.78 mm
- net N$6: track 1.58 -> 6.26 mm
- net N$7: track 1.72 -> 5.78 mm
- net SCL: track 0.00 -> 3.70 mm
- net MOSI: track 3.18 -> 0.00 mm
- net LED1: track 0.69 -> 2.36 mm
- net LED: track 0.59 -> 2.13 mm
- net N$2: track 9.78 -> 8.47 mm
- net FILTEROUT: track 19.5 -> 18.2 mm
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
Commit message: -a
a*
Parts:
- added R13: 0, rcl:0204/5
- moved R8 18.6 mm to (27.0, 32.0)
- moved C11 4.78 mm to (10.6, 22.3)
- moved U$4 3.36 mm to (4.59, 16.4), turned to 0 degrees
- moved BATT 1.76 mm to (5.01, 20.7)
- moved C2 1.54 mm to (16.2, 10.3)
- moved R3 1.54 mm to (23.4, 8.72)
- moved LED3 1.54 mm to (20.7, 4.62)
- moved R5 1.54 mm to (9.91, 5.14)
- moved CH1 1.54 mm to (14.5, 6.79)
- moved R4 1.54 mm to (22.8, 6.21)
- moved C3 1.54 mm to (10.0, 8.32)
- moved LED4 1.54 mm to (25.2, 4.62)
- moved X1 0.05 mm to (4.81, 5.58)
Connections:
- net MOSI: now also R13.1, R13.2
- net RESET: now also ISP.6; no longer ISP.5
- net VCC: now also ISP.5; no longer ISP.6
Routing:
- net GND: track 137.1 -> 181.2 mm
- net RESET: track 1.75 -> 27.4 mm
- net VCC: track 98.8 -> 109.4 mm
- net MOSI: track 0.00 -> 6.60 mm
- net V_BATT: track 22.8 -> 19.1 mm
- net MISO: track 18.8 -> 22.3 mm
- net CS: track 6.33 -> 8.87 mm
- net 3.3V: track 0.00 -> 2.54 mm
- net V_USB: track 33.0 -> 34.5 mm
- net SCK: track 21.4 -> 22.3 mm

Commit message: -a
a*
Parts:
- removed BATT: (no value), pinhead:1X02
- added BAT+, BAT-: (no value), 7_segment_lib:2,54/1,0
- moved R13 54.7 mm to (47.6, 25.0), turned to 90 degrees
Connections:
- new net N1: R13.1, SV1.MOSI, SV1.MOSI@1
- net DAC_CS: now also U1.26
- net DAC_SCK: now also U1.25
- net DAC_SDI: now also U1.24
- net GND: now also BAT-.1; no longer BATT.2
- net MOSI: no longer R13.1, SV1.MOSI, SV1.MOSI@1
- net VCC: now also U$4.NO; no longer U$4.COM
- net V_BATT: now also BAT+.1, U$4.COM; no longer BATT.1, U$4.NO
Routing:
- net VCC: track 109.4 -> 98.0 mm
- net V_BATT: track 19.1 -> 9.59 mm
- net MOSI: track 6.60 -> 12.5 mm
- net N1: track 0.00 -> 5.66 mm
- net GND: track 181.2 -> 177.6 mm
- net DAC_CS: track 0.00 -> 3.30 mm
- net DAC_SDI: track 0.00 -> 3.30 mm
- net DAC_SCK: track 0.00 -> 3.30 mm
- net SCK: track 22.3 -> 24.9 mm
Changed lines of the file:
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@@
 </autorouter>
 <elements>
-<element name="BATT" library="pinhead" library_urn="urn:adsk.eagle:library:325" package="1X02" package3d_urn="urn:adsk.eagle:package:22435/2" value="" x="5.0097" y="20.6964" smashed="yes" rot="R90">
-<attribute name="NAME" x="3.1809" y="18.0802" size="1.27" layer="25" ratio="10" rot="R90"/>
-<attribute name="VALUE" x="8.1847" y="18.1564" size="1.27" layer="27" rot="R90"/>
-</element>
 <element name="C1" library="rcl" library_urn="urn:adsk.eagle:library:334" package="C0603" package3d_urn="urn:adsk.eagle:package:23616/2" value="100n" x="28.264" y="21.3485" smashed="yes" rot="MR180">
 <attribute name="NAME" x="24.835" y="19.6975" size="1.27" layer="26" ratio="10" rot="MR180"/>
@@
 <attribute name="VALUE" x="26.8224" y="6.5278" size="1.27" layer="27" ratio="10" rot="R90"/>
 </element>
-<element name="R13" library="rcl" library_urn="urn:adsk.eagle:library:334" package="0204/5" package3d_urn="urn:adsk.eagle:package:23488/1" value="0" x="2.1844" y="-5.3848" smashed="yes">
-<attribute name="NAME" x="0.1778" y="-4.2164" size="0.9906" layer="25" ratio="10"/>
-<attribute name="SPICEPREFIX" value="R" x="2.1844" y="-5.3848" size="1.778" layer="27" display="off"/>
-<attribute name="VALUE" x="0.0508" y="-7.6962" size="0.9906" layer="27" ratio="10"/>
+<element name="R13" library="rcl" library_urn="urn:adsk.eagle:library:334" package="0204/5" package3d_urn="urn:adsk.eagle:package:23488/1" value="0" x="47.5996" y="25.0444" smashed="yes" rot="R90">
+<attribute name="NAME" x="46.4312" y="23.0378" size="0.9906" layer="25" ratio="10" rot="R90"/>
+<attribute name="SPICEPREFIX" value="R" x="47.5996" y="25.0444" size="1.778" layer="27" rot="R90" display="off"/>
+<attribute name="VALUE" x="49.911" y="22.9108" size="0.9906" layer="27" ratio="10" rot="R90"/>
+</element>
+<element name="BAT+" library="7_segment_lib" library_urn="urn:adsk.eagle:library:1964360" package="2,54/1,0" package3d_urn="urn:adsk.eagle:package:1964566/3" value="" x="0.6604" y="-6.1468" smashed="yes">
+<attribute name="NAME" x="-0.6096" y="-4.6228" size="1.27" layer="25" ratio="10"/>
+<attribute name="VALUE" x="0.6604" y="-5.1468" size="0.0254" layer="27"/>
+</element>
+<element name="BAT-" library="7_segment_lib" library_urn="urn:adsk.eagle:library:1964360" package="2,54/1,0" package3d_urn="urn:adsk.eagle:package:1964566/3" value="" x="0.6604" y="-10.8712" smashed="yes">
+<attribute name="NAME" x="-0.6096" y="-9.3472" size="1.27" layer="25" ratio="10"/>
+<attribute name="VALUE" x="0.6604" y="-9.8712" size="0.0254" layer="27"/>
 </element>
 </elements>
@@
 <contactref element="UART" pad="1"/>
 <contactref element="ISP" pad="1"/>
-<contactref element="BATT" pad="2"/>
 <contactref element="CH1" pad="3"/>
 <contactref element="CH1" pad="9"/>
@@
 <wire x1="10.6067" y1="21.441" x2="10.19445" y2="21.02875" width="0.6096" layer="16"/>
 <wire x1="10.19445" y1="21.02875" x2="8.27625" y2="21.02875" width="0.6096" layer="16"/>
-<wire x1="8.27625" y1="21.02875" x2="5.94735" y2="21.02875" width="0.6096" layer="16"/>
-<wire x1="5.94735" y1="21.02875" x2="5.0097" y2="21.9664" width="0.6096" layer="16"/>
 <wire x1="10.6067" y1="21.441" x2="11.1794" y2="21.441" width="0.6096" layer="16"/>
 <wire x1="24.6504" y1="24.7904" x2="26.85" y2="26.99" width="0.6096" layer="16"/>
@@
 <wire x1="7.6318" y1="3.9835" x2="9.602" y2="3.9835" width="0.6096" layer="16"/>
 <wire x1="9.602" y1="3.9835" x2="9.9122" y2="4.2937" width="0.6096" layer="16"/>
+<contactref element="BAT-" pad="1"/>
 <wire x1="34.3189" y1="36.397" x2="39.84875" y2="34.05" width="0" layer="19" extent="16-16"/>
 <wire x1="26.85" y1="26.99" x2="22.81" y2="35.43" width="0" layer="19" extent="16-16"/>
 <wire x1="15.3022" y1="10.26545" x2="16.5608" y2="13.9192" width="0" layer="19" extent="16-16"/>
+<wire x1="0.6604" y1="-10.8712" x2="7.2318" y2="3.9835" width="0" layer="19" extent="16-16"/>
 </signal>
 <signal name="V_BATT">
 <contactref element="C2" pad="1"/>
-<contactref element="BATT" pad="1"/>
 <contactref element="CH1" pad="5"/>
-<contactref element="U$4" pad="NO"/>
 <wire x1="17.2642" y1="8.6997" x2="17.2642" y2="10.00345" width="0.6096" layer="16"/>
 <wire x1="17.2642" y1="10.00345" x2="17.0022" y2="10.26545" width="0.6096" layer="16"/>
-<wire x1="7.134" y1="16.3896" x2="7.134" y2="17.3021" width="0.6096" layer="16"/>
-<wire x1="7.134" y1="17.3021" x2="5.0097" y2="19.4264" width="0.6096" layer="16"/>
-<wire x1="7.134" y1="16.3896" x2="11.0776" y2="12.446" width="0.6096" layer="16"/>
 <wire x1="16.0528" y1="12.446" x2="17.0688" y2="11.43" width="0.6096" layer="16"/>
 <wire x1="17.0688" y1="11.43" x2="17.0688" y2="10.19885" width="0.6096" layer="16"/>
 <wire x1="17.0688" y1="10.19885" x2="17.2642" y2="10.00345" width="0.6096" layer="16"/>
 <wire x1="11.0776" y1="12.446" x2="16.0528" y2="12.446" width="0.6096" layer="16"/>
+<contactref element="U$4" pad="COM"/>
+<contactref element="BAT+" pad="1"/>
+<wire x1="4.594" y1="16.3896" x2="11.0776" y2="12.446" width="0" layer="19" extent="16-16"/>
+<wire x1="0.6604" y1="-6.1468" x2="11.0776" y2="12.446" width="0" layer="19" extent="16-16"/>
 </signal>
 <signal name="LED">
@@
 <wire x1="34.47" y1="26.2868" x2="36.6268" y2="24.13" width="0.6096" layer="16"/>
 <wire x1="36.6268" y1="24.13" x2="48.8188" y2="24.13" width="0.6096" layer="16"/>
-<wire x1="50.6625" y1="25.1725" x2="53.2025" y2="25.1725" width="0" layer="19" extent="1-1"/>
+<wire x1="50.6625" y1="25.1725" x2="53.2025" y2="25.1725" width="0.6096" layer="16"/>
 </signal>
 <signal name="MOSI">
 <contactref element="ISP" pad="2"/>
 <contactref element="U1" pad="17"/>
-<contactref element="SV1" pad="MOSI"/>
-<contactref element="SV1" pad="MOSI@1"/>
-<wire x1="50.6625" y1="22.6325" x2="53.2025" y2="22.6325" width="0.6096" layer="16"/>
-<wire x1="39.55" y1="26.99" x2="39.55" y2="31.054" width="0.6096" layer="16"/>
-<contactref element="R13" pad="1"/>
+<wire x1="39.55" y1="26.99" x2="39.55" y2="28.6004" width="0.6096" layer="16"/>
 <contactref element="R13" pad="2"/>
-<wire x1="39.55" y1="26.99" x2="50.6625" y2="22.6325" width="0" layer="19" extent="1-1"/>
-<wire x1="4.7244" y1="-5.3848" x2="39.55" y2="26.99" width="0" layer="19" extent="1-1"/>
-<wire x1="-0.3556" y1="-5.3848" x2="4.7244" y2="-5.3848" width="0" layer="19" extent="1-1"/>
+<wire x1="39.55" y1="28.6004" x2="39.55" y2="31.054" width="0.6096" layer="16"/>
+<wire x1="39.55" y1="28.6004" x2="46.5836" y2="28.6004" width="0.6096" layer="16"/>
+<wire x1="46.5836" y1="28.6004" x2="47.5996" y2="27.5844" width="0.6096" layer="16"/>
 </signal>
 <signal name="CS">
@@
 <signal name="DAC_CS">
 <contactref element="U$2" pad="2"/>
+<contactref element="U1" pad="26"/>
+<wire x1="16.65" y1="30.27" x2="16.65" y2="27.03" width="0.6096" layer="16"/>
+<wire x1="16.65" y1="27.03" x2="16.69" y2="26.99" width="0.6096" layer="16"/>
 </signal>
 <signal name="DAC_SCK">
 <contactref element="U$2" pad="3"/>
+<contactref element="U1" pad="25"/>
+<wire x1="19.19" y1="30.27" x2="19.19" y2="27.03" width="0.6096" layer="16"/>
+<wire x1="19.19" y1="27.03" x2="19.23" y2="26.99" width="0.6096" layer="16"/>
 </signal>
 <signal name="DAC_SDI">
 <contactref element="U$2" pad="4"/>
+<contactref element="U1" pad="24"/>
+<wire x1="21.73" y1="30.27" x2="21.73" y2="27.03" width="0.6096" layer="16"/>
+<wire x1="21.73" y1="27.03" x2="21.77" y2="26.99" width="0.6096" layer="16"/>
 </signal>
 <signal name="PB7(XTAL2/TOSC2)">
@@
 <wire x1="14.11" y1="31.325" x2="16.65" y2="33.865" width="0.6096" layer="16"/>
 <wire x1="19.19" y1="33.865" x2="26.924" y2="33.865" width="0.6096" layer="16"/>
-<contactref element="U$4" pad="COM"/>
 <wire x1="26.924" y1="33.865" x2="27.455" y2="33.865" width="0.6096" layer="16"/>
 <wire x1="50.6625" y1="17.5525" x2="48.89" y2="15.78" width="0.6096" layer="16"/>
@@
 <wire x1="10.6067" y1="23.141" x2="10.17895" y2="23.56875" width="0.6096" layer="16"/>
 <wire x1="10.17895" y1="23.56875" x2="8.27625" y2="23.56875" width="0.6096" layer="16"/>
-<wire x1="4.594" y1="16.3896" x2="2.4384" y2="18.5452" width="0.6096" layer="16"/>
-<wire x1="2.4384" y1="22.9616" x2="3.302" y2="23.8252" width="0.6096" layer="16"/>
-<wire x1="3.302" y1="23.8252" x2="5.9436" y2="23.8252" width="0.6096" layer="16"/>
 <wire x1="5.9436" y1="23.8252" x2="8.0198" y2="23.8252" width="0.6096" layer="16"/>
 <wire x1="8.0198" y1="23.8252" x2="8.27625" y2="23.56875" width="0.6096" layer="16"/>
-<wire x1="2.4384" y1="18.5452" x2="2.4384" y2="22.9616" width="0.6096" layer="16"/>
 <wire x1="5.8315" y1="29.6567" x2="5.8315" y2="23.9373" width="0.6096" layer="16"/>
 <wire x1="5.8315" y1="23.9373" x2="5.9436" y2="23.8252" width="0.6096" layer="16"/>
@@
 <wire x1="29.9444" y1="24.712" x2="31.93" y2="24.712" width="0.6096" layer="16"/>
 <wire x1="27.414" y1="22.1816" x2="29.9444" y2="24.712" width="0.6096" layer="16"/>
+<contactref element="U$4" pad="NO"/>
 <wire x1="36.9191" y1="35.3951" x2="36.9191" y2="35.447" width="0" layer="19" extent="16-16"/>
+<wire x1="7.134" y1="16.3896" x2="8.27625" y2="23.56875" width="0" layer="19" extent="1-1"/>
 </signal>
 <signal name="N$2">
@@
 <wire x1="25.1714" y1="7.7651" x2="24.2118" y2="8.7247" width="0.6096" layer="16"/>
 </signal>
+<signal name="N1">
+<contactref element="SV1" pad="MOSI"/>
+<contactref element="SV1" pad="MOSI@1"/>
+<contactref element="R13" pad="1"/>
+<wire x1="50.6625" y1="22.6325" x2="53.2025" y2="22.6325" width="0.6096" layer="16"/>
+<wire x1="50.6625" y1="22.6325" x2="47.7277" y2="22.6325" width="0.6096" layer="16"/>
+<wire x1="47.7277" y1="22.6325" x2="47.5996" y2="22.5044" width="0.6096" layer="16"/>
+</signal>
 </signals>
