File: WaveP/main.brd (EAGLE design)
At the start: 57 x 45 mm, 48 parts, among them Q1 16MHz, U1 328P, U2 MCP6291T, X1 MINI-USB_SHIELD5P2-32005-601, X2 1503_09

Commit message: -a
a*
Parts:
- moved BAT- 45.4 mm to (2.54, 34.4)
- moved BAT+ 25.7 mm to (2.39, 19.5)
Connections:
- net GND: now also X1.M1, X1.M2
Routing:
- net GND: track 177.6 -> 212.7 mm
- net V_BATT: track 9.59 -> 21.7 mm
- net VCC: track 98.0 -> 106.1 mm
- added copper zone on layer 16, net GND
Changed lines of the file:
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@@
 <attribute name="VALUE" x="49.911" y="22.9108" size="0.9906" layer="27" ratio="10" rot="R90"/>
 </element>
-<element name="BAT+" library="7_segment_lib" library_urn="urn:adsk.eagle:library:1964360" package="2,54/1,0" package3d_urn="urn:adsk.eagle:package:1964566/3" value="" x="0.6604" y="-6.1468" smashed="yes">
-<attribute name="NAME" x="-0.6096" y="-4.6228" size="1.27" layer="25" ratio="10"/>
-<attribute name="VALUE" x="0.6604" y="-5.1468" size="0.0254" layer="27"/>
+<element name="BAT+" library="7_segment_lib" library_urn="urn:adsk.eagle:library:1964360" package="2,54/1,0" package3d_urn="urn:adsk.eagle:package:1964566/3" value="" x="2.3876" y="19.4564" smashed="yes">
+<attribute name="NAME" x="1.1176" y="20.9804" size="1.27" layer="25" ratio="10"/>
+<attribute name="VALUE" x="2.3876" y="20.4564" size="0.0254" layer="27"/>
 </element>
-<element name="BAT-" library="7_segment_lib" library_urn="urn:adsk.eagle:library:1964360" package="2,54/1,0" package3d_urn="urn:adsk.eagle:package:1964566/3" value="" x="0.6604" y="-10.8712" smashed="yes">
-<attribute name="NAME" x="-0.6096" y="-9.3472" size="1.27" layer="25" ratio="10"/>
-<attribute name="VALUE" x="0.6604" y="-9.8712" size="0.0254" layer="27"/>
+<element name="BAT-" library="7_segment_lib" library_urn="urn:adsk.eagle:library:1964360" package="2,54/1,0" package3d_urn="urn:adsk.eagle:package:1964566/3" value="" x="2.54" y="34.4424" smashed="yes">
+<attribute name="NAME" x="1.27" y="35.9664" size="1.27" layer="25" ratio="10"/>
+<attribute name="VALUE" x="2.54" y="35.4424" size="0.0254" layer="27"/>
 </element>
 </elements>
@@
 <wire x1="9.602" y1="3.9835" x2="9.9122" y2="4.2937" width="0.6096" layer="16"/>
 <contactref element="BAT-" pad="1"/>
+<wire x1="16.65" y1="35.565" x2="3.6626" y2="35.565" width="0.6096" layer="16"/>
+<wire x1="3.6626" y1="35.565" x2="2.54" y2="34.4424" width="0.6096" layer="16"/>
+<wire x1="53.2025" y1="30.2525" x2="55.4228" y2="28.0322" width="0.6096" layer="16"/>
+<wire x1="54.6873" y1="12.4725" x2="53.2025" y2="12.4725" width="0.6096" layer="16"/>
+<wire x1="55.4228" y1="28.0322" x2="55.4228" y2="13.208" width="0.6096" layer="16"/>
+<wire x1="55.4228" y1="13.208" x2="54.6873" y2="12.4725" width="0.6096" layer="16"/>
+<polygon width="0.2032" layer="16" isolate="1.016">
+<vertex x="0" y="45.0088"/>
+<vertex x="56.9976" y="45.0088"/>
+<vertex x="56.9976" y="0"/>
+<vertex x="0" y="0"/>
+</polygon>
+<contactref element="X1" pad="M1"/>
+<contactref element="X1" pad="M2"/>
+<wire x1="6.4318" y1="4.7835" x2="2.5818" y2="9.2335" width="0" layer="19" extent="1-1"/>
+<wire x1="16.5608" y1="13.9192" x2="15.3022" y2="10.26545" width="0" layer="19" extent="16-16"/>
+<wire x1="2.5818" y1="1.9335" x2="6.4318" y2="4.7835" width="0" layer="19" extent="1-1"/>
 <wire x1="34.3189" y1="36.397" x2="39.84875" y2="34.05" width="0" layer="19" extent="16-16"/>
-<wire x1="26.85" y1="26.99" x2="22.81" y2="35.43" width="0" layer="19" extent="16-16"/>
-<wire x1="15.3022" y1="10.26545" x2="16.5608" y2="13.9192" width="0" layer="19" extent="16-16"/>
-<wire x1="0.6604" y1="-10.8712" x2="7.2318" y2="3.9835" width="0" layer="19" extent="16-16"/>
 </signal>
 <signal name="V_BATT">
@@
 <wire x1="17.2642" y1="8.6997" x2="17.2642" y2="10.00345" width="0.6096" layer="16"/>
 <wire x1="17.2642" y1="10.00345" x2="17.0022" y2="10.26545" width="0.6096" layer="16"/>
-<wire x1="16.0528" y1="12.446" x2="17.0688" y2="11.43" width="0.6096" layer="16"/>
+<wire x1="17.0688" y1="11.43" x2="16.0528" y2="12.446" width="0.6096" layer="16"/>
 <wire x1="17.0688" y1="11.43" x2="17.0688" y2="10.19885" width="0.6096" layer="16"/>
 <wire x1="17.0688" y1="10.19885" x2="17.2642" y2="10.00345" width="0.6096" layer="16"/>
-<wire x1="11.0776" y1="12.446" x2="16.0528" y2="12.446" width="0.6096" layer="16"/>
 <contactref element="U$4" pad="COM"/>
 <contactref element="BAT+" pad="1"/>
-<wire x1="4.594" y1="16.3896" x2="11.0776" y2="12.446" width="0" layer="19" extent="16-16"/>
-<wire x1="0.6604" y1="-6.1468" x2="11.0776" y2="12.446" width="0" layer="19" extent="16-16"/>
+<wire x1="4.594" y1="16.3896" x2="4.594" y2="17.25" width="0.6096" layer="16"/>
+<wire x1="4.594" y1="17.25" x2="2.3876" y2="19.4564" width="0.6096" layer="16"/>
+<wire x1="8.5376" y1="12.446" x2="4.594" y2="16.3896" width="0.6096" layer="16"/>
+<wire x1="16.0528" y1="12.446" x2="8.5376" y2="12.446" width="0.6096" layer="16"/>
 </signal>
 <signal name="LED">
@@
 <wire x1="27.414" y1="22.1816" x2="29.9444" y2="24.712" width="0.6096" layer="16"/>
 <contactref element="U$4" pad="NO"/>
+<wire x1="7.134" y1="16.3896" x2="5.8315" y2="17.6921" width="0.6096" layer="16"/>
+<wire x1="5.8315" y1="17.6921" x2="5.8315" y2="23.9373" width="0.6096" layer="16"/>
 <wire x1="36.9191" y1="35.3951" x2="36.9191" y2="35.447" width="0" layer="19" extent="16-16"/>
-<wire x1="7.134" y1="16.3896" x2="8.27625" y2="23.56875" width="0" layer="19" extent="1-1"/>
 </signal>
 <signal name="N$2">
