File: WaveP/main.sch (EAGLE design)
At the start: 43 parts, among them Q1 16MHz, U1 328P, U2 MCP6291T, X1 MINI-USB_SHIELD5P2-32005-601, X2 1503_09

Commit message: -a
a
Parts:
- added C13: 100u, rcl:CPOL-USE2-5
Connections:
- new net N$10: C13.-, OUT.1, X2.2, X2.3
- net N$2: now also C13.+; no longer OUT.1
Changed lines of the file:
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@@
 <part name="SUPPLY18" library="SparkFun-PowerSymbols" library_urn="urn:adsk.eagle:library:530" deviceset="VCC" device=""/>
 <part name="GND26" library="SparkFun-PowerSymbols" library_urn="urn:adsk.eagle:library:530" deviceset="GND" device=""/>
+<part name="C13" library="rcl" library_urn="urn:adsk.eagle:library:334" deviceset="CPOL-US" device="E2-5" package3d_urn="urn:adsk.eagle:package:23346/2" value="100u"/>
 </parts>
 <sheets>
@@
 <instance part="GND26" gate="1" x="182.88" y="2.54" smashed="yes">
 <attribute name="VALUE" x="182.88" y="2.286" size="1.778" layer="96" align="top-center"/>
+</instance>
+<instance part="C13" gate="G$1" x="208.28" y="17.78" smashed="yes" rot="R90">
+<attribute name="NAME" x="207.645" y="18.796" size="1.778" layer="95" rot="R90"/>
+<attribute name="VALUE" x="212.471" y="18.796" size="1.778" layer="96" rot="R90"/>
 </instance>
 </instances>
@@
 <wire x1="190.5" y1="27.94" x2="205.74" y2="27.94" width="0.1524" layer="91"/>
 <wire x1="205.74" y1="27.94" x2="205.74" y2="17.78" width="0.1524" layer="91"/>
-<pinref part="OUT" gate="G$1" pin="1"/>
-<wire x1="226.06" y1="5.08" x2="205.74" y2="5.08" width="0.1524" layer="91"/>
-<wire x1="205.74" y1="5.08" x2="205.74" y2="17.78" width="0.1524" layer="91"/>
+<pinref part="C13" gate="G$1" pin="+"/>
 <junction x="205.74" y="17.78"/>
 </segment>
@@
 </segment>
 </net>
+<net name="N$10" class="0">
+<segment>
+<pinref part="X2" gate="G$1" pin="3"/>
+<wire x1="223.52" y1="25.4" x2="218.44" y2="25.4" width="0.1524" layer="91"/>
+<wire x1="218.44" y1="25.4" x2="218.44" y2="17.78" width="0.1524" layer="91"/>
+<wire x1="218.44" y1="17.78" x2="220.98" y2="17.78" width="0.1524" layer="91"/>
+<pinref part="X2" gate="G$1" pin="2"/>
+<wire x1="220.98" y1="17.78" x2="223.52" y2="17.78" width="0.1524" layer="91"/>
+<pinref part="C13" gate="G$1" pin="-"/>
+<wire x1="218.44" y1="17.78" x2="213.36" y2="17.78" width="0.1524" layer="91"/>
+<junction x="218.44" y="17.78"/>
+<pinref part="OUT" gate="G$1" pin="1"/>
+<wire x1="226.06" y1="5.08" x2="218.44" y2="5.08" width="0.1524" layer="91"/>
+<wire x1="218.44" y1="5.08" x2="218.44" y2="17.78" width="0.1524" layer="91"/>
+</segment>
+</net>

Commit message: -a
a
Parts:
- removed POT: 10k, con-lstb:MA03-1
- added TM1: (no value), adafruit:TRIMPOT3386
- C13: device rcl:CPOL-USE2-5 -> rcl:CPOL-USE2,5-6E
Connections:
- net BTN_NEXT: now also U1.PD7(AIN1); no longer U1.PD6(AIN0)
- net BTN_OK: now also U1.PD6(AIN0); no longer U1.PD7(AIN1)
- net FILTEROUT: now also TM1.E; no longer POT.3
- net GND: now also TM1.A; no longer POT.1
- net N$11: now also TM1.S; no longer POT.2
- net VCC: now also U$4.COM; no longer U$4.NO
- net V_BATT: now also U$4.NO; no longer U$4.COM

Commit message: -a
a
Connections:
- net LED: now also U1.PD3(INT1); no longer U1.PB0(ICP)
- net LED1: now also U1.PD4(XCK/T0); no longer U1.PB1(OC1A)
Changed lines of the file:
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@@
 <net name="LED" class="0">
-<segment>
-<pinref part="U1" gate="G$1" pin="PB0(ICP)"/>
-<wire x1="50.8" y1="2.54" x2="55.88" y2="2.54" width="0.1524" layer="91"/>
-<label x="55.88" y="2.54" size="1.27" layer="95" xref="yes"/>
-</segment>
 <segment>
 <pinref part="R1" gate="G$1" pin="1"/>
@@
 <label x="53.34" y="-35.56" size="1.27" layer="95" rot="R90" xref="yes"/>
 </segment>
+<segment>
+<pinref part="U1" gate="G$1" pin="PD3(INT1)"/>
+<wire x1="50.8" y1="17.78" x2="55.88" y2="17.78" width="0.1524" layer="91"/>
+<label x="55.88" y="17.78" size="1.27" layer="95" xref="yes"/>
+</segment>
 </net>
 <net name="LED1" class="0">
-<segment>
-<pinref part="U1" gate="G$1" pin="PB1(OC1A)"/>
-<wire x1="50.8" y1="0" x2="55.88" y2="0" width="0.1524" layer="91"/>
-<label x="55.88" y="0" size="1.27" layer="95" xref="yes"/>
-</segment>
 <segment>
 <pinref part="R2" gate="G$1" pin="1"/>
@@
 <label x="60.96" y="-35.56" size="1.27" layer="95" rot="R90" xref="yes"/>
 </segment>
+<segment>
+<pinref part="U1" gate="G$1" pin="PD4(XCK/T0)"/>
+<wire x1="50.8" y1="15.24" x2="55.88" y2="15.24" width="0.1524" layer="91"/>
+<label x="55.88" y="15.24" size="1.27" layer="95" xref="yes"/>
+</segment>
 </net>

Commit message: -a
a
Parts:
- removed U$1, U$3: BICOLOR_LED, 7_segment_lib:BICOLOR_LED
- added LED1, LED2, LED3, LED4: (no value), adafruit:LED3MM
Connections:
- net CS: now also U1.PB0(ICP); no longer U1.PB2(SS/OC1B)
- net GND: now also R1.2, R2.2, U2.V-; no longer U$1.C1, U$1.C2, U2.V+
- net LED: now also LED1.A; no longer R1.1
- net LED1: now also LED2.A; no longer R2.1
- net N$3: now also LED3.C, R4.1; no longer R3.2, U$3.A2
- net N$4: now also LED4.C, R3.1; no longer R4.2, U$3.A1
- net N$6: now also R4.2; no longer U$3.C2
- net N$7: now also R3.2; no longer U$3.C1
- net N$8: now also LED2.C, R2.1; no longer R1.2, U$1.A1
- net N$9: now also LED1.C, R1.1; no longer R2.2, U$1.A2
- net VCC: now also U2.V+; no longer U2.V-
- net V_USB: now also LED3.A, LED4.A; no longer R3.1, R4.1
Other:
- moved on the sheet: R1, R2, R3, R4

Commit message: -a
a*
Parts:
- added R13: 0, rcl:R-US_0204/5
Connections:
- net MOSI: now also R13.1, R13.2
- net RESET: now also ISP.6; no longer ISP.5
- net VCC: now also ISP.5; no longer ISP.6
Changed lines of the file:
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@@
 <part name="GND15" library="SparkFun-PowerSymbols" library_urn="urn:adsk.eagle:library:530" deviceset="GND" device=""/>
 <part name="SUPPLY12" library="SparkFun-PowerSymbols" library_urn="urn:adsk.eagle:library:530" deviceset="V_USB" device=""/>
-<part name="R3" library="rcl" library_urn="urn:adsk.eagle:library:334" deviceset="R-US_" device="R0603" package3d_urn="urn:adsk.eagle:package:23555/2" value="470"/>
-<part name="R4" library="rcl" library_urn="urn:adsk.eagle:library:334" deviceset="R-US_" device="R0603" package3d_urn="urn:adsk.eagle:package:23555/2" value="470"/>
-<part name="R5" library="rcl" library_urn="urn:adsk.eagle:library:334" deviceset="R-US_" device="R0603" package3d_urn="urn:adsk.eagle:package:23555/2" value="1.2k"/>
+<part name="R3" library="rcl" library_urn="urn:adsk.eagle:library:334" deviceset="R-US_" device="R0603" package3d_urn="urn:adsk.eagle:package:23555/3" value="470"/>
+<part name="R4" library="rcl" library_urn="urn:adsk.eagle:library:334" deviceset="R-US_" device="R0603" package3d_urn="urn:adsk.eagle:package:23555/3" value="470"/>
+<part name="R5" library="rcl" library_urn="urn:adsk.eagle:library:334" deviceset="R-US_" device="R0603" package3d_urn="urn:adsk.eagle:package:23555/3" value="1.2k"/>
 <part name="SUPPLY13" library="SparkFun-PowerSymbols" library_urn="urn:adsk.eagle:library:530" deviceset="V_USB" device=""/>
 <part name="C3" library="rcl" library_urn="urn:adsk.eagle:library:334" deviceset="C-US" device="C0603" package3d_urn="urn:adsk.eagle:package:23616/2" value="100n"/>
 <part name="GND16" library="SparkFun-PowerSymbols" library_urn="urn:adsk.eagle:library:530" deviceset="GND" device=""/>
 <part name="SUPPLY14" library="SparkFun-PowerSymbols" library_urn="urn:adsk.eagle:library:530" deviceset="V_USB" device=""/>
-<part name="R6" library="rcl" library_urn="urn:adsk.eagle:library:334" deviceset="R-US_" device="R0603" package3d_urn="urn:adsk.eagle:package:23555/2" value="1.5k"/>
+<part name="R6" library="rcl" library_urn="urn:adsk.eagle:library:334" deviceset="R-US_" device="R0603" package3d_urn="urn:adsk.eagle:package:23555/3" value="1.5k"/>
 <part name="C4" library="rcl" library_urn="urn:adsk.eagle:library:334" deviceset="C-US" device="C0603" package3d_urn="urn:adsk.eagle:package:23616/2" value="10n"/>
-<part name="R7" library="rcl" library_urn="urn:adsk.eagle:library:334" deviceset="R-US_" device="R0603" package3d_urn="urn:adsk.eagle:package:23555/2" value="100k"/>
-<part name="R8" library="rcl" library_urn="urn:adsk.eagle:library:334" deviceset="R-US_" device="R0603" package3d_urn="urn:adsk.eagle:package:23555/2" value="22k"/>
+<part name="R7" library="rcl" library_urn="urn:adsk.eagle:library:334" deviceset="R-US_" device="R0603" package3d_urn="urn:adsk.eagle:package:23555/3" value="100k"/>
+<part name="R8" library="rcl" library_urn="urn:adsk.eagle:library:334" deviceset="R-US_" device="R0603" package3d_urn="urn:adsk.eagle:package:23555/3" value="22k"/>
 <part name="Q1" library="crystal" library_urn="urn:adsk.eagle:library:204" deviceset="CRYSTAL" device="HC49S" package3d_urn="urn:adsk.eagle:package:12071/1" value="16MHz"/>
 <part name="C6" library="rcl" library_urn="urn:adsk.eagle:library:334" deviceset="C-US" device="C0603" package3d_urn="urn:adsk.eagle:package:23616/2" value="22p"/>
@@
 <part name="S1" library="SparkFun-Switches" library_urn="urn:adsk.eagle:library:535" deviceset="MOMENTARY-SWITCH-SPST" device="-PTH-6.0MM" package3d_urn="urn:adsk.eagle:package:40163/1"/>
 <part name="S2" library="SparkFun-Switches" library_urn="urn:adsk.eagle:library:535" deviceset="MOMENTARY-SWITCH-SPST" device="-PTH-6.0MM" package3d_urn="urn:adsk.eagle:package:40163/1"/>
-<part name="R9" library="rcl" library_urn="urn:adsk.eagle:library:334" deviceset="R-US_" device="R0603" package3d_urn="urn:adsk.eagle:package:23555/2" value="10k"/>
-<part name="R10" library="rcl" library_urn="urn:adsk.eagle:library:334" deviceset="R-US_" device="R0603" package3d_urn="urn:adsk.eagle:package:23555/2" value="10k"/>
-<part name="R11" library="rcl" library_urn="urn:adsk.eagle:library:334" deviceset="R-US_" device="R0603" package3d_urn="urn:adsk.eagle:package:23555/2" value="1k"/>
-<part name="R12" library="rcl" library_urn="urn:adsk.eagle:library:334" deviceset="R-US_" device="R0603" package3d_urn="urn:adsk.eagle:package:23555/2" value="1k"/>
+<part name="R9" library="rcl" library_urn="urn:adsk.eagle:library:334" deviceset="R-US_" device="R0603" package3d_urn="urn:adsk.eagle:package:23555/3" value="10k"/>
+<part name="R10" library="rcl" library_urn="urn:adsk.eagle:library:334" deviceset="R-US_" device="R0603" package3d_urn="urn:adsk.eagle:package:23555/3" value="10k"/>
+<part name="R11" library="rcl" library_urn="urn:adsk.eagle:library:334" deviceset="R-US_" device="R0603" package3d_urn="urn:adsk.eagle:package:23555/3" value="1k"/>
+<part name="R12" library="rcl" library_urn="urn:adsk.eagle:library:334" deviceset="R-US_" device="R0603" package3d_urn="urn:adsk.eagle:package:23555/3" value="1k"/>
 <part name="C8" library="rcl" library_urn="urn:adsk.eagle:library:334" deviceset="C-US" device="C0603" package3d_urn="urn:adsk.eagle:package:23616/2" value="100n"/>
 <part name="C9" library="rcl" library_urn="urn:adsk.eagle:library:334" deviceset="C-US" device="C0603" package3d_urn="urn:adsk.eagle:package:23616/2" value="100n"/>
@@
 <part name="C12" library="rcl" library_urn="urn:adsk.eagle:library:334" deviceset="C-US" device="C0603" package3d_urn="urn:adsk.eagle:package:23616/2" value="100n"/>
 <part name="GND23" library="SparkFun-PowerSymbols" library_urn="urn:adsk.eagle:library:530" deviceset="GND" device=""/>
-<part name="R1" library="rcl" library_urn="urn:adsk.eagle:library:334" deviceset="R-US_" device="R0603" package3d_urn="urn:adsk.eagle:package:23555/2" value="1k"/>
-<part name="R2" library="rcl" library_urn="urn:adsk.eagle:library:334" deviceset="R-US_" device="R0603" package3d_urn="urn:adsk.eagle:package:23555/2" value="1k"/>
+<part name="R1" library="rcl" library_urn="urn:adsk.eagle:library:334" deviceset="R-US_" device="R0603" package3d_urn="urn:adsk.eagle:package:23555/3" value="1k"/>
+<part name="R2" library="rcl" library_urn="urn:adsk.eagle:library:334" deviceset="R-US_" device="R0603" package3d_urn="urn:adsk.eagle:package:23555/3" value="1k"/>
 <part name="SV1" library="7_segment_lib" library_urn="urn:adsk.eagle:library:1964360" deviceset="SD_CARD" device="" package3d_urn="urn:adsk.eagle:package:8335/1"/>
 <part name="SV2" library="7_segment_lib" library_urn="urn:adsk.eagle:library:1964360" deviceset="OLED" device="" package3d_urn="urn:adsk.eagle:package:8635748/1"/>
@@
 <part name="GND25" library="SparkFun-PowerSymbols" library_urn="urn:adsk.eagle:library:530" deviceset="GND" device=""/>
 <part name="SUPPLY19" library="SparkFun-PowerSymbols" library_urn="urn:adsk.eagle:library:530" deviceset="VCC" device=""/>
+<part name="R13" library="rcl" library_urn="urn:adsk.eagle:library:334" deviceset="R-US_" device="0204/5" package3d_urn="urn:adsk.eagle:package:23488/1" value="0"/>
 </parts>
 <sheets>
@@
 <instance part="SUPPLY19" gate="G$1" x="195.58" y="30.48" smashed="yes">
 <attribute name="VALUE" x="195.58" y="33.274" size="1.778" layer="96" align="bottom-center"/>
+</instance>
+<instance part="R13" gate="G$1" x="-38.1" y="7.62" smashed="yes">
+<attribute name="NAME" x="-41.91" y="9.1186" size="1.778" layer="95"/>
+<attribute name="VALUE" x="-41.91" y="4.318" size="1.778" layer="96"/>
 </instance>
 </instances>
@@
 <net name="MOSI" class="0">
 <segment>
-<wire x1="-53.34" y1="7.62" x2="-48.26" y2="7.62" width="0.1524" layer="91"/>
-<label x="-48.26" y="7.62" size="1.27" layer="95" xref="yes"/>
 <pinref part="SV1" gate="G$1" pin="MOSI"/>
 <pinref part="SV1" gate="G$1" pin="MOSI@1"/>
-<wire x1="-53.34" y1="7.62" x2="-68.58" y2="7.62" width="0.1524" layer="91"/>
-<junction x="-53.34" y="7.62"/>
+<wire x1="-43.18" y1="7.62" x2="-68.58" y2="7.62" width="0.1524" layer="91"/>
+<pinref part="R13" gate="G$1" pin="1"/>
+<junction x="-43.18" y="7.62"/>
+<wire x1="-43.18" y1="7.62" x2="-53.34" y2="7.62" width="0.1524" layer="91"/>
 </segment>
 <segment>
@@
 <wire x1="50.8" y1="-5.08" x2="55.88" y2="-5.08" width="0.1524" layer="91"/>
 <label x="55.88" y="-5.08" size="1.27" layer="95" xref="yes"/>
+</segment>
+<segment>
+<pinref part="R13" gate="G$1" pin="2"/>
+<wire x1="-33.02" y1="7.62" x2="-30.48" y2="7.62" width="0.1524" layer="91"/>
+<label x="-30.48" y="7.62" size="1.27" layer="95" xref="yes"/>
 </segment>
 </net>
@@
 <net name="RESET" class="0">
 <segment>
-<pinref part="ISP" gate="1" pin="5"/>
-<wire x1="-81.28" y1="30.48" x2="-86.36" y2="30.48" width="0.1524" layer="91"/>
+<pinref part="ISP" gate="1" pin="6"/>
+<wire x1="-81.28" y1="30.48" x2="-86.36" y2="33.02" width="0.1524" layer="91"/>
 <label x="-81.28" y="30.48" size="1.27" layer="95" xref="yes"/>
 </segment>
@@
 </segment>
 <segment>
-<pinref part="ISP" gate="1" pin="6"/>
-<wire x1="-86.36" y1="33.02" x2="-83.82" y2="33.02" width="0.1524" layer="91"/>
+<pinref part="ISP" gate="1" pin="5"/>
+<wire x1="-86.36" y1="30.48" x2="-83.82" y2="33.02" width="0.1524" layer="91"/>
 <wire x1="-83.82" y1="33.02" x2="-83.82" y2="35.56" width="0.1524" layer="91"/>
 <pinref part="SUPPLY8" gate="G$1" pin="VCC"/>

Commit message: -a
a*
Parts:
- removed BATT: (no value), pinhead:PINHD-1X2
- added BAT+, BAT-: (no value), 7_segment_lib:2,54/1,0
Connections:
- new net N1: R13.1, SV1.MOSI, SV1.MOSI@1
- net DAC_CS: now also U1.PC3(ADC3)
- net DAC_SCK: now also U1.PC2(ADC2)
- net DAC_SDI: now also U1.PC1(ADC1)
- net GND: now also BAT-.P; no longer BATT.2
- net MOSI: no longer R13.1, SV1.MOSI, SV1.MOSI@1
- net VCC: now also U$4.NO; no longer U$4.COM
- net V_BATT: now also BAT+.P, U$4.COM; no longer BATT.1, U$4.NO
Changed lines of the file:
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@@
 <parts>
 <part name="U1" library="SparkFun-IC-Microcontroller" library_urn="urn:adsk.eagle:library:525" deviceset="ATMEGA328P_PDIP" device="" package3d_urn="urn:adsk.eagle:package:38942/1" value="328P"/>
-<part name="BATT" library="pinhead" library_urn="urn:adsk.eagle:library:325" deviceset="PINHD-1X2" device="" package3d_urn="urn:adsk.eagle:package:22435/2"/>
 <part name="ISP" library="con-lstb" library_urn="urn:adsk.eagle:library:162" deviceset="MA06-1" device="" package3d_urn="urn:adsk.eagle:package:8340/1"/>
 <part name="UART" library="con-lstb" library_urn="urn:adsk.eagle:library:162" deviceset="MA03-1" device="" package3d_urn="urn:adsk.eagle:package:8339/1"/>
@@
 <part name="C13" library="rcl" library_urn="urn:adsk.eagle:library:334" deviceset="CPOL-US" device="E2,5-6E" package3d_urn="urn:adsk.eagle:package:23430/1" value="100u"/>
 <part name="TM1" library="adafruit" library_urn="urn:adsk.eagle:library:420" deviceset="TRIMPOT" device="3386" package3d_urn="urn:adsk.eagle:package:6240934/1"/>
-<part name="SUPPLY20" library="SparkFun-PowerSymbols" library_urn="urn:adsk.eagle:library:530" deviceset="VCC" device=""/>
-<part name="SUPPLY21" library="SparkFun-PowerSymbols" library_urn="urn:adsk.eagle:library:530" deviceset="V_BATT" device=""/>
 <part name="LED1" library="adafruit" library_urn="urn:adsk.eagle:library:420" deviceset="LED" device="3MM" package3d_urn="urn:adsk.eagle:package:6240537/1"/>
 <part name="LED2" library="adafruit" library_urn="urn:adsk.eagle:library:420" deviceset="LED" device="3MM" package3d_urn="urn:adsk.eagle:package:6240537/1"/>
@@
 <part name="SUPPLY19" library="SparkFun-PowerSymbols" library_urn="urn:adsk.eagle:library:530" deviceset="VCC" device=""/>
 <part name="R13" library="rcl" library_urn="urn:adsk.eagle:library:334" deviceset="R-US_" device="0204/5" package3d_urn="urn:adsk.eagle:package:23488/1" value="0"/>
+<part name="SUPPLY20" library="SparkFun-PowerSymbols" library_urn="urn:adsk.eagle:library:530" deviceset="VCC" device=""/>
+<part name="SUPPLY21" library="SparkFun-PowerSymbols" library_urn="urn:adsk.eagle:library:530" deviceset="V_BATT" device=""/>
+<part name="BAT+" library="7_segment_lib" library_urn="urn:adsk.eagle:library:1964360" deviceset="2,54/1,0" device="" package3d_urn="urn:adsk.eagle:package:1964566/3"/>
+<part name="BAT-" library="7_segment_lib" library_urn="urn:adsk.eagle:library:1964360" deviceset="2,54/1,0" device="" package3d_urn="urn:adsk.eagle:package:1964566/3"/>
 </parts>
 <sheets>
@@
 <attribute name="VALUE" x="7.62" y="-15.24" size="1.778" layer="96"/>
 </instance>
-<instance part="BATT" gate="G$1" x="-55.88" y="55.88" smashed="yes">
-<attribute name="NAME" x="-62.23" y="61.595" size="1.778" layer="95"/>
-<attribute name="VALUE" x="-62.23" y="50.8" size="1.778" layer="96"/>
-</instance>
 <instance part="ISP" gate="1" x="-93.98" y="27.94" smashed="yes">
 <attribute name="VALUE" x="-95.25" y="15.24" size="1.778" layer="96"/>
@@
 <attribute name="VALUE" x="173.99" y="3.81" size="1.778" layer="96" rot="R90"/>
 </instance>
-<instance part="SUPPLY20" gate="G$1" x="-48.26" y="58.42" smashed="yes">
-<attribute name="VALUE" x="-48.26" y="61.214" size="1.778" layer="96" align="bottom-center"/>
-</instance>
-<instance part="SUPPLY21" gate="G$1" x="-33.02" y="55.88" smashed="yes">
-<attribute name="VALUE" x="-33.02" y="58.674" size="1.778" layer="96" align="bottom-center"/>
-</instance>
 <instance part="LED1" gate="G$1" x="53.34" y="-50.8" smashed="yes">
 <attribute name="NAME" x="56.896" y="-55.372" size="1.778" layer="95" rot="R90"/>
@@
 <attribute name="NAME" x="-41.91" y="9.1186" size="1.778" layer="95"/>
 <attribute name="VALUE" x="-41.91" y="4.318" size="1.778" layer="96"/>
+</instance>
+<instance part="SUPPLY20" gate="G$1" x="-33.02" y="55.88" smashed="yes">
+<attribute name="VALUE" x="-33.02" y="58.674" size="1.778" layer="96" align="bottom-center"/>
+</instance>
+<instance part="SUPPLY21" gate="G$1" x="-48.26" y="58.42" smashed="yes">
+<attribute name="VALUE" x="-48.26" y="61.214" size="1.778" layer="96" align="bottom-center"/>
+</instance>
+<instance part="BAT+" gate="P" x="-55.88" y="58.42" smashed="yes" rot="R180">
+<attribute name="NAME" x="-57.277" y="61.6458" size="1.778" layer="95" rot="R180"/>
+<attribute name="VALUE" x="-54.737" y="61.722" size="1.778" layer="96" rot="R180"/>
+</instance>
+<instance part="BAT-" gate="P" x="-55.88" y="55.88" smashed="yes" rot="R180">
+<attribute name="NAME" x="-57.277" y="54.0258" size="1.778" layer="95" rot="R180"/>
+<attribute name="VALUE" x="-54.737" y="59.182" size="1.778" layer="96" rot="R180"/>
 </instance>
 </instances>
@@
 </segment>
 <segment>
-<pinref part="BATT" gate="G$1" pin="2"/>
 <pinref part="GND1" gate="1" pin="GND"/>
 <wire x1="-58.42" y1="55.88" x2="-68.58" y2="55.88" width="0.1524" layer="91"/>
+<pinref part="BAT-" gate="P" pin="P"/>
 </segment>
 <segment>
@@
 </segment>
 <segment>
-<pinref part="BATT" gate="G$1" pin="1"/>
 <pinref part="SUPPLY1" gate="G$1" pin="V_BATT"/>
 <wire x1="-58.42" y1="58.42" x2="-68.58" y2="58.42" width="0.1524" layer="91"/>
 <wire x1="-68.58" y1="58.42" x2="-68.58" y2="60.96" width="0.1524" layer="91"/>
+<pinref part="BAT+" gate="P" pin="P"/>
 </segment>
 <segment>
@@
 </segment>
 <segment>
-<pinref part="U$4" gate="G$1" pin="NO"/>
-<wire x1="-38.1" y1="55.88" x2="-33.02" y2="55.88" width="0.1524" layer="91"/>
+<pinref part="U$4" gate="G$1" pin="COM"/>
+<wire x1="-48.26" y1="58.42" x2="-45.72" y2="58.42" width="0.1524" layer="91"/>
 <pinref part="SUPPLY21" gate="G$1" pin="V_BATT"/>
 </segment>
@@
 <net name="MOSI" class="0">
 <segment>
-<pinref part="SV1" gate="G$1" pin="MOSI"/>
-<pinref part="SV1" gate="G$1" pin="MOSI@1"/>
-<wire x1="-43.18" y1="7.62" x2="-68.58" y2="7.62" width="0.1524" layer="91"/>
-<pinref part="R13" gate="G$1" pin="1"/>
-<junction x="-43.18" y="7.62"/>
-<wire x1="-43.18" y1="7.62" x2="-53.34" y2="7.62" width="0.1524" layer="91"/>
-</segment>
-<segment>
 <pinref part="ISP" gate="1" pin="2"/>
 <wire x1="-86.36" y1="22.86" x2="-81.28" y2="22.86" width="0.1524" layer="91"/>
@@
 <label x="101.6" y="17.78" size="1.27" layer="95" rot="R180" xref="yes"/>
 </segment>
+<segment>
+<pinref part="U1" gate="G$1" pin="PC3(ADC3)"/>
+<wire x1="50.8" y1="40.64" x2="55.88" y2="40.64" width="0.1524" layer="91"/>
+<label x="55.88" y="40.64" size="1.27" layer="95" xref="yes"/>
+</segment>
 </net>
 <net name="DAC_SCK" class="0">
@@
 <label x="101.6" y="15.24" size="1.27" layer="95" rot="R180" xref="yes"/>
 </segment>
+<segment>
+<pinref part="U1" gate="G$1" pin="PC2(ADC2)"/>
+<wire x1="50.8" y1="43.18" x2="55.88" y2="43.18" width="0.1524" layer="91"/>
+<label x="55.88" y="43.18" size="1.27" layer="95" xref="yes"/>
+</segment>
 </net>
 <net name="DAC_SDI" class="0">
@@
 <wire x1="109.22" y1="12.7" x2="101.6" y2="12.7" width="0.1524" layer="91"/>
 <label x="101.6" y="12.7" size="1.27" layer="95" rot="R180" xref="yes"/>
+</segment>
+<segment>
+<pinref part="U1" gate="G$1" pin="PC1(ADC1)"/>
+<wire x1="50.8" y1="45.72" x2="55.88" y2="45.72" width="0.1524" layer="91"/>
+<label x="55.88" y="45.72" size="1.27" layer="95" xref="yes"/>
 </segment>
 </net>
@@
 </segment>
 <segment>
-<pinref part="U$4" gate="G$1" pin="COM"/>
-<wire x1="-48.26" y1="58.42" x2="-45.72" y2="58.42" width="0.1524" layer="91"/>
-<pinref part="SUPPLY20" gate="G$1" pin="VCC"/>
-</segment>
-<segment>
 <pinref part="U2" gate="G$1" pin="V+"/>
 <wire x1="195.58" y1="25.4" x2="195.58" y2="30.48" width="0.1524" layer="91"/>
 <pinref part="SUPPLY19" gate="G$1" pin="VCC"/>
+</segment>
+<segment>
+<pinref part="U$4" gate="G$1" pin="NO"/>
+<wire x1="-38.1" y1="55.88" x2="-33.02" y2="55.88" width="0.1524" layer="91"/>
+<pinref part="SUPPLY20" gate="G$1" pin="VCC"/>
 </segment>
 </net>
@@
 </segment>
 </net>
+<net name="N1" class="0">
+<segment>
+<pinref part="SV1" gate="G$1" pin="MOSI"/>
+<pinref part="SV1" gate="G$1" pin="MOSI@1"/>
+<wire x1="-43.18" y1="7.62" x2="-68.58" y2="7.62" width="0.1524" layer="91"/>
+<pinref part="R13" gate="G$1" pin="1"/>
+<junction x="-43.18" y="7.62"/>
+<wire x1="-43.18" y1="7.62" x2="-53.34" y2="7.62" width="0.1524" layer="91"/>
+</segment>
+</net>
