File: WaveP/main.sch (EAGLE design)
At the start: 48 parts, among them Q1 16MHz, U1 328P, U2 MCP6291T, X1 MINI-USB_SHIELD5P2-32005-601, X2 1503_09

Commit message: -a
a*
Connections:
- net GND: now also X1S.S1, X1S.S2
Changed lines of the file:
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@@
 <attribute name="VALUE" x="-54.737" y="59.182" size="1.778" layer="96" rot="R180"/>
+</instance>
+<instance part="X1" gate="S" x="-114.3" y="-10.16" smashed="yes">
+<attribute name="NAME" x="-113.03" y="-11.43" size="1.778" layer="95"/>
 </instance>
 </instances>
@@
 <wire x1="-106.68" y1="-15.24" x2="-109.22" y2="-15.24" width="0.1524" layer="91"/>
 <junction x="-109.22" y="-15.24"/>
+<pinref part="X1" gate="S" pin="S1"/>
+<wire x1="-116.84" y1="-12.7" x2="-114.3" y2="-12.7" width="0.1524" layer="91"/>
+<junction x="-109.22" y="-12.7"/>
+<wire x1="-114.3" y1="-12.7" x2="-109.22" y2="-12.7" width="0.1524" layer="91"/>
+<wire x1="-114.3" y1="-12.7" x2="-109.22" y2="-12.7" width="0.1524" layer="91"/>
+<junction x="-114.3" y="-12.7"/>
+<pinref part="X1" gate="S" pin="S2"/>
 </segment>
 <segment>

Commit message: -a
a*
Parts:
- removed BAT+, BAT-: (no value), 7_segment_lib:2,54/1,0
- added BAT: (no value), pinhead:PINHD-1X2
Connections:
- net GND: now also BAT.2; no longer BAT-.P
- net V_BATT: now also BAT.1; no longer BAT+.P
Changed lines of the file:
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@@
 <part name="SUPPLY20" library="SparkFun-PowerSymbols" library_urn="urn:adsk.eagle:library:530" deviceset="VCC" device=""/>
 <part name="SUPPLY21" library="SparkFun-PowerSymbols" library_urn="urn:adsk.eagle:library:530" deviceset="V_BATT" device=""/>
-<part name="BAT+" library="7_segment_lib" library_urn="urn:adsk.eagle:library:1964360" deviceset="2,54/1,0" device="" package3d_urn="urn:adsk.eagle:package:1964566/3"/>
-<part name="BAT-" library="7_segment_lib" library_urn="urn:adsk.eagle:library:1964360" deviceset="2,54/1,0" device="" package3d_urn="urn:adsk.eagle:package:1964566/3"/>
+<part name="BAT" library="pinhead" library_urn="urn:adsk.eagle:library:325" deviceset="PINHD-1X2" device="" package3d_urn="urn:adsk.eagle:package:22435/2"/>
 </parts>
 <sheets>
@@
 <attribute name="VALUE" x="-48.26" y="61.214" size="1.778" layer="96" align="bottom-center"/>
 </instance>
-<instance part="BAT+" gate="P" x="-55.88" y="58.42" smashed="yes" rot="R180">
-<attribute name="NAME" x="-57.277" y="61.6458" size="1.778" layer="95" rot="R180"/>
-<attribute name="VALUE" x="-54.737" y="61.722" size="1.778" layer="96" rot="R180"/>
-</instance>
-<instance part="BAT-" gate="P" x="-55.88" y="55.88" smashed="yes" rot="R180">
-<attribute name="NAME" x="-57.277" y="54.0258" size="1.778" layer="95" rot="R180"/>
-<attribute name="VALUE" x="-54.737" y="59.182" size="1.778" layer="96" rot="R180"/>
-</instance>
 <instance part="X1" gate="S" x="-114.3" y="-10.16" smashed="yes">
 <attribute name="NAME" x="-113.03" y="-11.43" size="1.778" layer="95"/>
+</instance>
+<instance part="BAT" gate="G$1" x="-55.88" y="55.88" smashed="yes">
+<attribute name="NAME" x="-62.23" y="61.595" size="1.778" layer="95"/>
+<attribute name="VALUE" x="-62.23" y="50.8" size="1.778" layer="96"/>
 </instance>
 </instances>
@@
 <pinref part="GND1" gate="1" pin="GND"/>
 <wire x1="-58.42" y1="55.88" x2="-68.58" y2="55.88" width="0.1524" layer="91"/>
-<pinref part="BAT-" gate="P" pin="P"/>
+<pinref part="BAT" gate="G$1" pin="2"/>
 </segment>
 <segment>
@@
 <wire x1="-58.42" y1="58.42" x2="-68.58" y2="58.42" width="0.1524" layer="91"/>
 <wire x1="-68.58" y1="58.42" x2="-68.58" y2="60.96" width="0.1524" layer="91"/>
-<pinref part="BAT+" gate="P" pin="P"/>
-</segment>
-<segment>
+<pinref part="BAT" gate="G$1" pin="1"/>
+</segment>
+<segment>
