File: power_meter1/main1.sch (EAGLE design)
At the start: 41 parts, among them IC1 7805TV, Q1 16M, U1 LT1999CS8-50PBF, U2 ATMEGA168PA-AU, X1 SCREWTERM_5MM_4WAY

Commit message: a
Other:
- moved on the sheet: JP2, OK1, R1, R7
