File: Adafruit-USB-Isolator-PCB-master/Adafruit USB Isolator.sch (EAGLE design)
At the start: 28 parts, among them U1 ADuM4160, U2 ADuM5000, X2 05241, X3 06564

Commit message: a
Parts:
- removed FID1, FID2, FID3: FIDUCIAL"", microbuilder:FIDUCIAL""
- removed U$10, U$7, U$8, U$9: MOUNTINGHOLE2.5_THICK, microbuilder:MOUNTINGHOLE2.5_THICK
