File: oled/128x64_ada.brd (EAGLE design)
At the start: 38 x 28.5 mm, 36 parts, among them Q1 BSS138, Q2 BSS138, U1 UG-2864HSWEG01

Commit message: -ma
Parts:
- removed D1, D3: 1N4148, microbuilder:SOD-323
- removed FID1, FID2: FIDUCIAL"", microbuilder:FIDUCIAL_1MM
- removed JP1: (no value), microbuilder:1X08_ROUND_70
- removed R2, R4, R6: 10K, microbuilder:0805
- removed SJ1, SJ2: (no value), microbuilder:SOLDERJUMPER_REFLOW_NOPASTE
- removed U$23, U$24, U$25, U$26: MOUNTINGHOLE2.5, microbuilder:MOUNTINGHOLE_2.5_PLATED
- removed U$27: (no value), microbuilder:ADAFRUIT_2.5MM
- removed U$28: (no value), microbuilder:LOGIC_5VREADY_5MM
- removed U$3: (no value), microbuilder:ADAFRUIT_5MM
- removed U2: (no value), microbuilder:SOT23-5
- added SV1: (no value), con-lstb:MA06-1
- added U3: LM1117IMP-3.3, NSC_By_element14_Batch_1.1:SOT230P696X180-4N
- D2: value 1N4148 -> 1N456A; device microbuilder:SOD-323 -> Fairchild_By_element14_Batch_1:DIO_1N456A
- Q1, Q2: device microbuilder:SOT23-WIDE -> BeagleBone_Blue_R3:SOT323
- R11, R12, R13, R14, R5: device microbuilder:0805 -> microbuilder:0603
- moved R13 22.1 mm to (25.5, 27.0)
- moved Q1 19.2 mm to (22.4, 15.0), turned to 270 degrees
- moved Q2 18.5 mm to (18.4, 10.7), turned to 270 degrees
- moved C2 17.5 mm to (9.94, 3.76), turned to 0 degrees
- moved R12 17.5 mm to (20.9, 10.4), turned to 90 degrees
- moved C6 16.2 mm to (17.0, 3.08)
- moved R11 15.1 mm to (24.6, 15.1)
- moved R14 14.3 mm to (22.8, 26.8)
- moved C1 12.5 mm to (16.7, 26.3), turned to 180 degrees
- moved C7 11.5 mm to (14.0, 16.9), turned to 90 degrees
- moved C4 9.89 mm to (12.7, 11.3), turned to 0 degrees
- moved D2 8.71 mm to (16.5, 13.1), flipped to the top, turned to 180 degrees
- moved C3 7.40 mm to (8.91, 11.2)
- moved R5 7.30 mm to (16.5, 8.45), turned to 0 degrees
- moved R3 1.22 mm to (24.8, 10.3)
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Connections:
- net D0/SCLK/SCK_3.3V renamed SCK_3.3V
- removed net CS_3.3V: D1.A, R4.1, U1.13
- removed net CS_5.0V: D1.C, JP1.5
- removed net D0/SCLK/SCK_5.0V: JP1.2, Q2.3, R14.1
- removed net D1/MOSI/SDA1_3.3V: Q1.2, R11.1, SJ1.1, U1.19
- removed net D1/MOSI/SDA_5.0V: JP1.1, Q1.3, R13.1
- removed net DC/SA0_3.3V: D3.A, R6.1, U1.15
- removed net DC/SA0_5.0V: D3.C, JP1.3
- removed net N$1: R2.2, SJ2.2, U1.11
- removed net N$2: SJ1.2, U1.20
- new net SCK_5.0V: Q2.3, R14.1, SV1.5
- new net SDA_3.3V: Q1.2, R11.1, U1.19, U1.20
- new net SDA_5.0V: Q1.3, R13.1, SV1.6
- net 3.3V: now also SV1.1, U1.11, U3.2, U3.4; no longer JP1.6, R4.2, R6.2, SJ2.1, U2.5
- net GND: now also SV1.3, U1.15, U3.1; no longer JP1.8, R2.1, U2.2
- net RST_3.3V: now also D2.2; no longer D2.A
- net RST_5.0V: now also D2.1, SV1.4; no longer D2.C, JP1.4
- net VIN: now also SV1.2, U3.3; no longer JP1.7, U2.1, U2.3
Routing:
- net 3.3V: track 101.5 -> 22.1 mm
- net D1/MOSI/SDA1_3.3V: track 58.3 -> 0.00 mm, vias 2 -> 0
- net VIN: track 48.3 -> 6.34 mm, vias 2 -> 0
- net SCK_3.3V: track 39.5 -> 4.87 mm, vias 2 -> 0
- net DC/SA0_3.3V: track 28.9 -> 0.00 mm, vias 2 -> 0
- net N$1: track 28.8 -> 0.00 mm
- net D0/SCLK/SCK_5.0V: track 27.3 -> 0.00 mm
- net D1/MOSI/SDA_5.0V: track 24.4 -> 0.00 mm, vias 1 -> 0
- net CS_3.3V: track 23.3 -> 0.00 mm, vias 2 -> 0
- net N$2: track 20.6 -> 0.00 mm
- net RST_3.3V: track 20.1 -> 2.78 mm, vias 2 -> 0
- net SCK_5.0V: track 0.00 -> 15.3 mm
- net GND: track 41.2 -> 27.6 mm, vias 8 -> 0
- net SDA_5.0V: track 0.00 -> 12.5 mm
- net N$7: track 13.0 -> 5.71 mm
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- removed copper zone on layer 1, net GND
Other:
- board size 38 x 28.5 mm -> 38 x 29.3 mm
- board text removed: "3v3"
- board text removed: "CS"
- board text removed: "Clk"
- board text removed: "Close"
- board text removed: "DC"
- board text removed: "Data"
- board text removed: "For I2C"
- board text removed: "Gnd"
- board text removed: "Rst"
- board text removed: "SA0"
- board text removed: "SJ1"
- board text removed: "SJ1/2"
- board text removed: "SJ2"
- board text removed: "SSD1306 0.96" 128x64 OLED"
- board text removed: "Vin"
- board text removed: "v2.1"
