File: oled/128x64_ada.sch (EAGLE design)
At the start: 33 parts, among them Q1 BSS138, Q2 BSS138, U1 UG-2864HSWEG01

Commit message: -ma
Parts:
- removed D1, D3: 1N4148, microbuilder:DIODESOD-323
- removed FID1, FID2: FIDUCIAL"", microbuilder:FIDUCIAL""
- removed JP1: (no value), microbuilder:HEADER-1X870MIL
- removed R2, R4, R6: 10K, microbuilder:RESISTOR0805
- removed SJ1, SJ2: (no value), microbuilder:SOLDERJUMPERREFLOW_NOPASTE
- removed U$23, U$24, U$25, U$26: MOUNTINGHOLE2.5, microbuilder:MOUNTINGHOLE2.5
- removed U2: (no value), microbuilder:VREG_SOT23-5
- added SV1: (no value), con-lstb:MA06-1
- added U3: LM1117IMP-3.3, NSC_By_element14_Batch_1.1:LM1117IMP-3.3
- D2: value 1N4148 -> 1N456A; device microbuilder:DIODESOD-323 -> Fairchild_By_element14_Batch_1:1N456A
- Q1, Q2: device microbuilder:MOSFET-NWIDE -> BeagleBone_Blue_R3:MOSFET-NCHANNEL2N7002PW
- R11, R12, R13, R14, R5: device microbuilder:RESISTOR0805 -> microbuilder:RESISTOR0603
Connections:
- net D0/SCLK/SCK_3.3V renamed SCK_3.3V
- removed net CS_3.3V: D1.A, R4.1, U1./CS
- removed net CS_5.0V: D1.C, JP1.5
- removed net D0/SCLK/SCK_5.0V: JP1.2, Q2.D, R14.1
- removed net D1/MOSI/SDA1_3.3V: Q1.S, R11.1, SJ1.1, U1.D1/SPI_SDIN/I2C_SDA
- removed net D1/MOSI/SDA_5.0V: JP1.1, Q1.D, R13.1
- removed net DC/SA0_3.3V: D3.A, R6.1, U1.DC/I2C_SA0
- removed net DC/SA0_5.0V: D3.C, JP1.3
- removed net N$1: R2.2, SJ2.2, U1.BS1
- removed net N$2: SJ1.2, U1.D2/I2C_SDA
- new net SCK_5.0V: Q2.D, R14.1, SV1.5
- new net SDA_3.3V: Q1.S, R11.1, U1.D1/SPI_SDIN/I2C_SDA, U1.D2/I2C_SDA
- new net SDA_5.0V: Q1.D, R13.1, SV1.6
- net 3.3V: now also SV1.1, U1.BS1, U3.VOUT, U3.VOUT_2; no longer JP1.6, R4.2, R6.2, SJ2.1, U2.OUT
- net GND: now also SV1.3, U1.DC/I2C_SA0, U3.ADJ/GND; no longer JP1.8, R2.1, U2.GND
- net RST_5.0V: now also SV1.4; no longer JP1.4
- net VIN: now also SV1.2, U3.VIN; no longer JP1.7, U2.EN, U2.IN
Other:
- note removed: "= 011110+SA0+RW"
- note removed: "= 0x7A with DC/SA0_5.0V floating/high"
- note removed: "Bus default = SPI4"
- note removed: "Close SJ2 for I2C"
- note removed: "Close for"
- note removed: "I2C"
- note removed: "ToDo: Change address to default low"
- moved on the sheet: C1, C2, C3, C4, C5, C6, C7, C8, R11, R12, R13, R14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
