File: CurrentProbe/main.brd (EAGLE design)
At the start: 160 x 100 mm, 15 parts, among them CN1 USB, J1 v+, J2 v-, U1 LT1999CS8-50PBF, X1 SMA-142-0701-801/806

Commit message: a
Parts:
- C1, C2, C4: device rcl:C050-030X075 -> rcl:C0805
- moved LED1 66.0 mm to (24.1, 45.1)
- moved U1 65.2 mm to (15.3, 41.3), turned to 180 degrees
- moved C3 63.6 mm to (12.6, 51.3), turned to 270 degrees
- moved R1 58.9 mm to (28.3, 42.3), turned to 90 degrees
- moved JP2 54.7 mm to (6.21, 51.0), turned to 90 degrees
- moved J2 54.3 mm to (29.2, 54.5)
- moved X1 53.3 mm to (0.82, 42.0)
- moved JP3 47.8 mm to (8.33, 41.8), turned to 270 degrees
- moved J1 46.0 mm to (29.2, 35.0)
- moved CN1 45.9 mm to (19.3, 51.8), turned to 180 degrees
- moved C4 44.7 mm to (10.3, 51.3), turned to 270 degrees
- moved FB1 43.0 mm to (18.4, 41.4), turned to 90 degrees
- moved C2 40.9 mm to (15.4, 45.0), turned to 180 degrees
- moved R2 38.9 mm to (21.1, 44.8), turned to 180 degrees
- moved C1 28.3 mm to (11.8, 46.8)
Routing:
- net GND: track 0.00 -> 22.0 mm
- net V-: track 0.00 -> 21.8 mm
- net V+: track 0.00 -> 16.0 mm
- net +5V: track 0.00 -> 12.5 mm
- net VCC: track 0.00 -> 11.9 mm
- net REF: track 0.00 -> 8.96 mm
- net OUT: track 0.00 -> 5.05 mm
- net OUTPUT: track 0.00 -> 5.01 mm
- net N$1: track 0.00 -> 2.29 mm
Other:
- board size 160 x 100 mm -> 161.3 x 101.3 mm

Commit message: a
Parts:
- removed CN1: USB, adafruit:USB-MINIB
- added X2: MINI-USB_SHIELD5P4-32005-400, con-cypressindustries:32005-400
Connections:
- net GND: no longer CN1.GND
- net VCC: no longer CN1.VBUS
Changed lines of the file:
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@@
 <attribute name="VALUE" x="7.212" y="54.846" size="1.27" layer="27" ratio="10" rot="R270"/>
-</element>
-<element name="CN1" library="adafruit" library_urn="urn:adsk.eagle:library:420" package="USB-MINIB" package3d_urn="urn:adsk.eagle:package:6240633/1" value="USB" x="19.3" y="51.83" smashed="yes" rot="R180">
-<attribute name="NAME" x="22.61" y="46.48" size="1.27" layer="25" rot="R180"/>
-<attribute name="VALUE" x="22.61" y="58.18" size="1.27" layer="27" rot="R180"/>
 </element>
 <element name="FB1" library="rcl" library_urn="urn:adsk.eagle:library:334" package="0204/7" package3d_urn="urn:adsk.eagle:package:23498/2" value="0" x="18.41" y="41.39" smashed="yes" rot="R90">
@@
 <attribute name="VALUE" x="2.09" y="33.095" size="1.778" layer="27"/>
 </element>
+<element name="X2" library="con-cypressindustries" library_urn="urn:adsk.eagle:library:138" package="32005-400" package3d_urn="urn:adsk.eagle:package:6462/1" value="MINI-USB_SHIELD5P4-32005-400" x="-13.97" y="6.35" smashed="yes">
+<attribute name="MF" value="" x="-13.97" y="6.35" size="1.778" layer="27" display="off"/>
+<attribute name="MPN" value="" x="-13.97" y="6.35" size="1.778" layer="27" display="off"/>
+<attribute name="NAME" x="-18.415" y="12.065" size="1.27" layer="25"/>
+<attribute name="OC_FARNELL" value="unknown" x="-13.97" y="6.35" size="1.778" layer="27" display="off"/>
+<attribute name="OC_NEWARK" value="unknown" x="-13.97" y="6.35" size="1.778" layer="27" display="off"/>
+<attribute name="POPULARITY" value="0" x="-13.97" y="6.35" size="1.778" layer="27" display="off"/>
+<attribute name="VALUE" x="-18.415" y="-0.635" size="1.27" layer="27"/>
+</element>
 </elements>
 <signals>
 <signal name="VCC">
-<contactref element="CN1" pad="VBUS"/>
 <contactref element="JP2" pad="2"/>
 <contactref element="R2" pad="2"/>
@@
 <wire x1="20.275" y1="44.755" x2="18.855" y2="44.755" width="0.8128" layer="1"/>
 <wire x1="18.855" y1="44.755" x2="18.41" y2="45.2" width="0.8128" layer="1"/>
-<wire x1="20.9" y1="47.766" x2="20.955" y2="47.711" width="0.4064" layer="1"/>
 <wire x1="20.275" y1="45.04" x2="20.275" y2="44.755" width="0.4064" layer="1"/>
 <wire x1="20.955" y1="47.711" x2="20.955" y2="45.72" width="0.4064" layer="1"/>
@@
 </signal>
 <signal name="GND">
-<contactref element="CN1" pad="GND"/>
 <contactref element="U1" pad="5"/>
 <contactref element="X1" pad="G@1"/>
@@
 <wire x1="12.725" y1="46.8" x2="12.725" y2="50.184" width="0.8128" layer="1"/>
 <wire x1="12.725" y1="50.184" x2="12.625" y2="50.284" width="0.8128" layer="1"/>
-<wire x1="17.7" y1="47.766" x2="24.09" y2="45.835" width="0" layer="19" extent="1-1"/>
-<wire x1="14.45" y1="44.99" x2="17.7" y2="47.766" width="0" layer="19" extent="1-1"/>
+<wire x1="14.45" y1="44.99" x2="24.09" y2="45.835" width="0" layer="19" extent="1-1"/>
 <wire x1="3.3854" y1="46.4046" x2="3.3854" y2="46.4046" width="0" layer="19" extent="1-16"/>
 <wire x1="3.3854" y1="37.5654" x2="3.3854" y2="46.4046" width="0" layer="19" extent="1-1"/>

Commit message: a
Connections:
- net GND: now also X2.5, X2.M1, X2.M2, X2.M3, X2.M4
- net VCC: now also X2.1
Changed lines of the file:
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@@
 <wire x1="10.26" y1="52.24" x2="10.25" y2="52.23" width="0.8128" layer="1"/>
 <wire x1="10.25" y1="52.23" x2="10.16" y2="52.23" width="0.8128" layer="1"/>
+<contactref element="X2" pad="1"/>
 <wire x1="12.625" y1="52.316" x2="18.41" y2="45.2" width="0" layer="19" extent="1-1"/>
+<wire x1="-10.97" y1="7.95" x2="18.41" y2="45.2" width="0" layer="19" extent="1-1"/>
 </signal>
 <signal name="GND">
@@
 <wire x1="12.725" y1="46.8" x2="12.725" y2="50.184" width="0.8128" layer="1"/>
 <wire x1="12.725" y1="50.184" x2="12.625" y2="50.284" width="0.8128" layer="1"/>
+<contactref element="X2" pad="5"/>
+<contactref element="X2" pad="M1"/>
+<contactref element="X2" pad="M2"/>
+<contactref element="X2" pad="M3"/>
+<contactref element="X2" pad="M4"/>
 <wire x1="14.45" y1="44.99" x2="24.09" y2="45.835" width="0" layer="19" extent="1-1"/>
 <wire x1="3.3854" y1="46.4046" x2="3.3854" y2="46.4046" width="0" layer="19" extent="1-16"/>
 <wire x1="3.3854" y1="37.5654" x2="3.3854" y2="46.4046" width="0" layer="19" extent="1-1"/>
 <wire x1="3.3854" y1="37.5654" x2="3.3854" y2="37.5654" width="0" layer="19" extent="1-16"/>
+<wire x1="-11.07" y1="10.8" x2="3.3854" y2="37.5654" width="0" layer="19" extent="1-1"/>
+<wire x1="-16.97" y1="10.8" x2="-11.07" y2="10.8" width="0" layer="19" extent="1-1"/>
+<wire x1="-10.97" y1="4.75" x2="-11.07" y2="10.8" width="0" layer="19" extent="1-1"/>
+<wire x1="-11.07" y1="1.9" x2="-10.97" y2="4.75" width="0" layer="19" extent="1-1"/>
+<wire x1="-16.97" y1="1.9" x2="-11.07" y2="1.9" width="0" layer="19" extent="1-1"/>
 </signal>
 <signal name="V+">

Commit message: a
Parts:
- moved X2 55.7 mm to (19.4, 51.0), turned to 270 degrees
Changed lines of the file:
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@@
 <setting verticaltext="up"/>
 </settings>
-<grid distance="25" unitdist="mil" unit="mil" style="dots" multiple="1" display="yes" altdistance="5" altunitdist="mil" altunit="mil"/>
+<grid distance="0.5" unitdist="mm" unit="mm" style="dots" multiple="1" display="yes" altdistance="5" altunitdist="mil" altunit="mil"/>
 <layers>
 <layer number="1" name="Top" color="4" fill="1" visible="yes" active="yes"/>
@@
 <attribute name="VALUE" x="2.09" y="33.095" size="1.778" layer="27"/>
 </element>
-<element name="X2" library="con-cypressindustries" library_urn="urn:adsk.eagle:library:138" package="32005-400" package3d_urn="urn:adsk.eagle:package:6462/1" value="MINI-USB_SHIELD5P4-32005-400" x="-13.97" y="6.35" smashed="yes">
-<attribute name="MF" value="" x="-13.97" y="6.35" size="1.778" layer="27" display="off"/>
-<attribute name="MPN" value="" x="-13.97" y="6.35" size="1.778" layer="27" display="off"/>
-<attribute name="NAME" x="-18.415" y="12.065" size="1.27" layer="25"/>
-<attribute name="OC_FARNELL" value="unknown" x="-13.97" y="6.35" size="1.778" layer="27" display="off"/>
-<attribute name="OC_NEWARK" value="unknown" x="-13.97" y="6.35" size="1.778" layer="27" display="off"/>
-<attribute name="POPULARITY" value="0" x="-13.97" y="6.35" size="1.778" layer="27" display="off"/>
-<attribute name="VALUE" x="-18.415" y="-0.635" size="1.27" layer="27"/>
+<element name="X2" library="con-cypressindustries" library_urn="urn:adsk.eagle:library:138" package="32005-400" package3d_urn="urn:adsk.eagle:package:6462/1" value="MINI-USB_SHIELD5P4-32005-400" x="19.35" y="50.97" smashed="yes" rot="R270">
+<attribute name="MF" value="" x="19.35" y="50.97" size="1.778" layer="27" rot="R270" display="off"/>
+<attribute name="MPN" value="" x="19.35" y="50.97" size="1.778" layer="27" rot="R270" display="off"/>
+<attribute name="NAME" x="25.065" y="55.415" size="1.27" layer="25" rot="R270"/>
+<attribute name="OC_FARNELL" value="unknown" x="19.35" y="50.97" size="1.778" layer="27" rot="R270" display="off"/>
+<attribute name="OC_NEWARK" value="unknown" x="19.35" y="50.97" size="1.778" layer="27" rot="R270" display="off"/>
+<attribute name="POPULARITY" value="0" x="19.35" y="50.97" size="1.778" layer="27" rot="R270" display="off"/>
+<attribute name="VALUE" x="12.365" y="55.415" size="1.27" layer="27" rot="R270"/>
 </element>
 </elements>
@@
 <contactref element="X2" pad="1"/>
 <wire x1="12.625" y1="52.316" x2="18.41" y2="45.2" width="0" layer="19" extent="1-1"/>
-<wire x1="-10.97" y1="7.95" x2="18.41" y2="45.2" width="0" layer="19" extent="1-1"/>
+<wire x1="20.95" y1="47.97" x2="18.41" y2="45.2" width="0" layer="19" extent="1-1"/>
 </signal>
 <signal name="GND">
@@
 <wire x1="3.3854" y1="37.5654" x2="3.3854" y2="46.4046" width="0" layer="19" extent="1-1"/>
 <wire x1="3.3854" y1="37.5654" x2="3.3854" y2="37.5654" width="0" layer="19" extent="1-16"/>
-<wire x1="-11.07" y1="10.8" x2="3.3854" y2="37.5654" width="0" layer="19" extent="1-1"/>
-<wire x1="-16.97" y1="10.8" x2="-11.07" y2="10.8" width="0" layer="19" extent="1-1"/>
-<wire x1="-10.97" y1="4.75" x2="-11.07" y2="10.8" width="0" layer="19" extent="1-1"/>
-<wire x1="-11.07" y1="1.9" x2="-10.97" y2="4.75" width="0" layer="19" extent="1-1"/>
-<wire x1="-16.97" y1="1.9" x2="-11.07" y2="1.9" width="0" layer="19" extent="1-1"/>
+<wire x1="23.8" y1="48.07" x2="3.3854" y2="37.5654" width="0" layer="19" extent="1-1"/>
+<wire x1="23.8" y1="53.97" x2="23.8" y2="48.07" width="0" layer="19" extent="1-1"/>
+<wire x1="17.75" y1="47.97" x2="23.8" y2="48.07" width="0" layer="19" extent="1-1"/>
+<wire x1="14.9" y1="48.07" x2="17.75" y2="47.97" width="0" layer="19" extent="1-1"/>
+<wire x1="14.9" y1="53.97" x2="14.9" y2="48.07" width="0" layer="19" extent="1-1"/>
 </signal>
 <signal name="V+">

Commit message: a
Routing:
- net GND: track 22.0 -> 45.3 mm
- net VCC: track 11.8 -> 17.0 mm
Changed lines of the file:
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@@
 <setting verticaltext="up"/>
 </settings>
-<grid distance="0.5" unitdist="mm" unit="mm" style="dots" multiple="1" display="yes" altdistance="5" altunitdist="mil" altunit="mil"/>
+<grid distance="25" unitdist="mil" unit="mil" style="dots" multiple="1" display="yes" altdistance="5" altunitdist="mil" altunit="mil"/>
 <layers>
 <layer number="1" name="Top" color="4" fill="1" visible="yes" active="yes"/>
@@
 <wire x1="10.25" y1="52.23" x2="10.16" y2="52.23" width="0.8128" layer="1"/>
 <contactref element="X2" pad="1"/>
-<wire x1="12.625" y1="52.316" x2="18.41" y2="45.2" width="0" layer="19" extent="1-1"/>
-<wire x1="20.95" y1="47.97" x2="18.41" y2="45.2" width="0" layer="19" extent="1-1"/>
+<wire x1="12.625" y1="52.316" x2="13.089" y2="52.316" width="0.8128" layer="1"/>
+<wire x1="13.089" y1="52.316" x2="13.97" y2="51.435" width="0.8128" layer="1"/>
+<wire x1="20.955" y1="51.435" x2="20.955" y2="47.975" width="0.4064" layer="1"/>
+<wire x1="20.955" y1="47.975" x2="20.95" y2="47.97" width="0.4064" layer="1"/>
+<wire x1="20.955" y1="47.711" x2="20.95" y2="47.97" width="0" layer="19" extent="1-1"/>
+<wire x1="13.97" y1="51.435" x2="20.955" y2="51.435" width="0" layer="19" extent="1-1"/>
 </signal>
 <signal name="GND">
@@
 <contactref element="X2" pad="M3"/>
 <contactref element="X2" pad="M4"/>
-<wire x1="14.45" y1="44.99" x2="24.09" y2="45.835" width="0" layer="19" extent="1-1"/>
+<wire x1="14.9" y1="53.97" x2="23.8" y2="53.97" width="0.8128" layer="1"/>
+<wire x1="14.45" y1="44.99" x2="14.45" y2="47.62" width="0.8128" layer="1"/>
+<wire x1="14.45" y1="47.62" x2="14.9" y2="48.07" width="0.8128" layer="1"/>
+<wire x1="23.8" y1="48.07" x2="23.8" y2="53.97" width="0.8128" layer="1"/>
+<wire x1="24.09" y1="45.835" x2="24.09" y2="47.78" width="0.6096" layer="1"/>
+<wire x1="24.09" y1="47.78" x2="23.8" y2="48.07" width="0.6096" layer="1"/>
+<wire x1="17.75" y1="47.97" x2="17.65" y2="48.07" width="0.508" layer="1"/>
+<wire x1="17.65" y1="48.07" x2="14.9" y2="48.07" width="0.508" layer="1"/>
+<wire x1="12.625" y1="50.284" x2="14.9" y2="53.97" width="0" layer="19" extent="1-1"/>
 <wire x1="3.3854" y1="46.4046" x2="3.3854" y2="46.4046" width="0" layer="19" extent="1-16"/>
 <wire x1="3.3854" y1="37.5654" x2="3.3854" y2="46.4046" width="0" layer="19" extent="1-1"/>
 <wire x1="3.3854" y1="37.5654" x2="3.3854" y2="37.5654" width="0" layer="19" extent="1-16"/>
-<wire x1="23.8" y1="48.07" x2="3.3854" y2="37.5654" width="0" layer="19" extent="1-1"/>
-<wire x1="23.8" y1="53.97" x2="23.8" y2="48.07" width="0" layer="19" extent="1-1"/>
-<wire x1="17.75" y1="47.97" x2="23.8" y2="48.07" width="0" layer="19" extent="1-1"/>
-<wire x1="14.9" y1="48.07" x2="17.75" y2="47.97" width="0" layer="19" extent="1-1"/>
-<wire x1="14.9" y1="53.97" x2="14.9" y2="48.07" width="0" layer="19" extent="1-1"/>
 </signal>
 <signal name="V+">

Commit message: a
Parts:
- moved LED1 21.4 mm to (3.17, 49.6), turned to 270 degrees
- moved R2 19.6 mm to (2.85, 51.9), turned to 90 degrees
Routing:
- net GND: track 45.3 -> 35.8 mm
- net VCC: track 17.0 -> 24.9 mm
- net REF: track 8.96 -> 5.53 mm
- net N$1: track 2.29 -> 1.65 mm
- added copper zone on layer 1, net GND
Changed lines of the file:
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@@
 <attribute name="VALUE" x="5.155" y="45.64" size="1.27" layer="27" rot="R270"/>
 </element>
-<element name="LED1" library="led" library_urn="urn:adsk.eagle:library:259" package="CHIP-LED0603" package3d_urn="urn:adsk.eagle:package:15819/3" value="yellow" x="24.09" y="45.085" smashed="yes">
-<attribute name="NAME" x="23.455" y="44.45" size="1.27" layer="25" rot="R90"/>
-<attribute name="POPULARITY" value="26" x="66" y="-0.635" size="1.778" layer="27" display="off"/>
-<attribute name="VALUE" x="25.995" y="44.45" size="1.27" layer="27" rot="R90"/>
+<element name="LED1" library="led" library_urn="urn:adsk.eagle:library:259" package="CHIP-LED0603" package3d_urn="urn:adsk.eagle:package:15819/3" value="yellow" x="3.175" y="49.57" smashed="yes" rot="R270">
+<attribute name="NAME" x="2.54" y="50.205" size="1.27" layer="25"/>
+<attribute name="POPULARITY" value="26" x="-42.545" y="7.66" size="1.778" layer="27" rot="R270" display="off"/>
+<attribute name="VALUE" x="2.54" y="47.665" size="1.27" layer="27"/>
 </element>
 <element name="R1" library="resistor" library_urn="urn:adsk.eagle:library:348" package="R2512" package3d_urn="urn:adsk.eagle:package:23545/2" value="10m" x="28.285" y="42.27" smashed="yes" rot="R90">
@@
 <attribute name="VALUE" x="31.46" y="39.73" size="1.27" layer="27" rot="R90"/>
 </element>
-<element name="R2" library="rcl" library_urn="urn:adsk.eagle:library:334" package="R0603" package3d_urn="urn:adsk.eagle:package:23555/3" value="470" x="21.125" y="44.755" smashed="yes" rot="R180">
-<attribute name="NAME" x="21.76" y="44.12" size="1.27" layer="25" rot="R180"/>
-<attribute name="POPULARITY" value="77" x="4.615" y="99.365" size="1.778" layer="27" rot="R180" display="off"/>
-<attribute name="SPICEPREFIX" value="R" x="4.615" y="99.365" size="1.778" layer="27" rot="R180" display="off"/>
-<attribute name="VALUE" x="21.76" y="46.66" size="1.27" layer="27" rot="R180"/>
+<element name="R2" library="rcl" library_urn="urn:adsk.eagle:library:334" package="R0603" package3d_urn="urn:adsk.eagle:package:23555/3" value="470" x="2.845" y="51.9" smashed="yes" rot="R90">
+<attribute name="NAME" x="2.21" y="51.265" size="1.27" layer="25" rot="R90"/>
+<attribute name="POPULARITY" value="77" x="57.455" y="68.41" size="1.778" layer="27" rot="R90" display="off"/>
+<attribute name="SPICEPREFIX" value="R" x="57.455" y="68.41" size="1.778" layer="27" rot="R90" display="off"/>
+<attribute name="VALUE" x="4.75" y="51.265" size="1.27" layer="27" rot="R90"/>
 </element>
 <element name="U1" library="LTC_By_element14_Batch_1" package="SOIC127P600X175-8N" value="LT1999CS8-50PBF" x="15.26" y="41.33" smashed="yes" rot="R180">
@@
 <contactref element="C3" pad="+"/>
 <contactref element="FB1" pad="2"/>
-<wire x1="20.275" y1="44.755" x2="18.855" y2="44.755" width="0.8128" layer="1"/>
 <wire x1="18.855" y1="44.755" x2="18.41" y2="45.2" width="0.8128" layer="1"/>
-<wire x1="20.275" y1="45.04" x2="20.275" y2="44.755" width="0.4064" layer="1"/>
 <wire x1="20.955" y1="47.711" x2="20.955" y2="45.72" width="0.4064" layer="1"/>
-<wire x1="20.955" y1="45.72" x2="20.275" y2="45.04" width="0.4064" layer="1"/>
 <wire x1="6.205" y1="52.23" x2="10.16" y2="52.23" width="0.8128" layer="1"/>
 <wire x1="10.16" y1="52.23" x2="12.539" y2="52.23" width="0.8128" layer="1"/>
@@
 <wire x1="20.955" y1="51.435" x2="20.955" y2="47.975" width="0.4064" layer="1"/>
 <wire x1="20.955" y1="47.975" x2="20.95" y2="47.97" width="0.4064" layer="1"/>
-<wire x1="20.955" y1="47.711" x2="20.95" y2="47.97" width="0" layer="19" extent="1-1"/>
-<wire x1="13.97" y1="51.435" x2="20.955" y2="51.435" width="0" layer="19" extent="1-1"/>
+<wire x1="13.97" y1="51.435" x2="20.32" y2="51.435" width="0.8128" layer="1"/>
+<wire x1="20.32" y1="51.435" x2="20.955" y2="51.435" width="0.4064" layer="1"/>
+<wire x1="2.845" y1="52.75" x2="5.685" y2="52.75" width="0.8128" layer="1"/>
+<wire x1="5.685" y1="52.75" x2="6.205" y2="52.23" width="0.8128" layer="1"/>
+<wire x1="20.95" y1="47.97" x2="20.955" y2="47.711" width="0" layer="19" extent="1-1"/>
+<wire x1="18.855" y1="44.755" x2="20.955" y2="45.72" width="0" layer="19" extent="1-1"/>
 </signal>
 <signal name="GND">
@@
 <wire x1="12.725" y1="46.8" x2="12.7962" y2="46.7288" width="0.508" layer="1"/>
 <wire x1="12.7962" y1="46.7288" x2="12.7962" y2="46.355" width="0.508" layer="1"/>
-<wire x1="12.7962" y1="46.355" x2="12.7962" y2="45.085" width="0.508" layer="1"/>
-<wire x1="12.7962" y1="45.085" x2="12.7962" y2="43.235" width="0.508" layer="1"/>
-<wire x1="12.8912" y1="44.99" x2="12.7962" y2="45.085" width="0.508" layer="1"/>
 <wire x1="12.625" y1="50.284" x2="12.7962" y2="50.1128" width="0.508" layer="1"/>
-<wire x1="14.45" y1="44.99" x2="12.8912" y2="44.99" width="0.8128" layer="1"/>
 <wire x1="12.725" y1="46.8" x2="12.7962" y2="46.7288" width="0.8128" layer="1"/>
-<wire x1="12.7962" y1="46.7288" x2="12.7962" y2="45.085" width="0.8128" layer="1"/>
 <wire x1="3.3854" y1="46.4046" x2="3.3854" y2="46.8704" width="0.8128" layer="1"/>
 <wire x1="3.3854" y1="46.8704" x2="6.205" y2="49.69" width="0.8128" layer="1"/>
@@
 <wire x1="12.625" y1="50.284" x2="10.316" y2="50.284" width="0.8128" layer="1"/>
 <wire x1="10.316" y1="50.284" x2="10.26" y2="50.34" width="0.8128" layer="1"/>
-<wire x1="12.725" y1="46.8" x2="12.725" y2="50.184" width="0.8128" layer="1"/>
 <wire x1="12.725" y1="50.184" x2="12.625" y2="50.284" width="0.8128" layer="1"/>
 <contactref element="X2" pad="5"/>
@@
 <wire x1="14.45" y1="47.62" x2="14.9" y2="48.07" width="0.8128" layer="1"/>
 <wire x1="23.8" y1="48.07" x2="23.8" y2="53.97" width="0.8128" layer="1"/>
-<wire x1="24.09" y1="45.835" x2="24.09" y2="47.78" width="0.6096" layer="1"/>
 <wire x1="24.09" y1="47.78" x2="23.8" y2="48.07" width="0.6096" layer="1"/>
 <wire x1="17.75" y1="47.97" x2="17.65" y2="48.07" width="0.508" layer="1"/>
 <wire x1="17.65" y1="48.07" x2="14.9" y2="48.07" width="0.508" layer="1"/>
-<wire x1="12.625" y1="50.284" x2="14.9" y2="53.97" width="0" layer="19" extent="1-1"/>
+<polygon width="0.4064" layer="1" isolate="1.27">
+<vertex x="-1.27" y="55.245"/>
+<vertex x="24.765" y="55.245"/>
+<vertex x="24.765" y="33.655"/>
+<vertex x="-1.27" y="33.655"/>
+</polygon>
+<wire x1="3.925" y1="49.57" x2="6.085" y2="49.57" width="0.8128" layer="1"/>
+<wire x1="6.085" y1="49.57" x2="6.205" y2="49.69" width="0.8128" layer="1"/>
+<wire x1="14.45" y1="44.99" x2="12.7962" y2="46.355" width="0" layer="19" extent="1-1"/>
 <wire x1="3.3854" y1="46.4046" x2="3.3854" y2="46.4046" width="0" layer="19" extent="1-16"/>
-<wire x1="3.3854" y1="37.5654" x2="3.3854" y2="46.4046" width="0" layer="19" extent="1-1"/>
+<wire x1="12.7962" y1="43.235" x2="14.45" y2="44.99" width="0" layer="19" extent="1-1"/>
+<wire x1="14.9" y1="53.97" x2="12.625" y2="50.284" width="0" layer="19" extent="1-1"/>
+<wire x1="3.3854" y1="37.5654" x2="3.3854" y2="46.4046" width="0" layer="19" extent="1-16"/>
 <wire x1="3.3854" y1="37.5654" x2="3.3854" y2="37.5654" width="0" layer="19" extent="1-16"/>
 </signal>
@@
 <wire x1="8.97" y1="44.37" x2="8.33" y2="44.37" width="0.508" layer="1"/>
 <wire x1="11.375" y1="41.965" x2="8.97" y2="44.37" width="0.508" layer="1"/>
-<wire x1="8.33" y1="44.37" x2="10.76" y2="46.8" width="0.8128" layer="1"/>
 <wire x1="10.76" y1="46.8" x2="10.825" y2="46.8" width="0.8128" layer="1"/>
+<wire x1="8.33" y1="44.37" x2="10.76" y2="46.8" width="0" layer="19" extent="1-1"/>
 </signal>
 <signal name="V-">
@@
 <contactref element="LED1" pad="A"/>
 <contactref element="R2" pad="1"/>
-<wire x1="24.09" y1="44.335" x2="22.395" y2="44.335" width="0.6096" layer="1"/>
-<wire x1="22.395" y1="44.335" x2="21.975" y2="44.755" width="0.6096" layer="1"/>
+<wire x1="2.425" y1="49.57" x2="2.425" y2="50.63" width="0.8128" layer="1"/>
+<wire x1="2.425" y1="50.63" x2="2.845" y2="51.05" width="0.8128" layer="1"/>
 </signal>
 </signals>

Commit message: a
Parts:
- moved X2 2.54 mm to (16.8, 51.0)
- moved C4 2.54 mm to (7.72, 51.3)
- moved JP2 2.54 mm to (3.67, 51.0)
- moved LED1 2.54 mm to (0.64, 49.6)
- moved R2 2.54 mm to (0.30, 51.9)
- moved C3 2.54 mm to (10.1, 51.3)
- moved C1 1.90 mm to (11.8, 44.9)
- moved FB1 0.64 mm to (19.0, 41.4)
- moved C2 0.63 mm to (16.0, 45.0)
Routing:
- net GND: track 35.8 -> 27.5 mm
- net VCC: track 24.9 -> 22.3 mm

Commit message: a
Parts:
- moved C4 10.7 mm to (16.4, 45.0), turned to 180 degrees
- moved C2 7.73 mm to (14.8, 37.4)
- moved R2 5.75 mm to (6.02, 52.5)
- moved LED1 5.44 mm to (6.07, 49.8), turned to 180 degrees
- moved J1 4.13 mm to (25.1, 35.0)
- moved J2 4.13 mm to (25.1, 54.5)
- moved R1 4.13 mm to (24.2, 42.3)
- moved C3 1.27 mm to (8.81, 51.3)
- moved X2 1.27 mm to (15.5, 51.0)
- moved JP2 0.64 mm to (3.03, 51.0)
Routing:
- net GND: track 27.5 -> 54.0 mm
- net V-: track 21.8 -> 17.7 mm
- net V+: track 16.0 -> 11.9 mm
- net VCC: track 22.3 -> 23.9 mm
- net +5V: track 12.5 -> 13.9 mm
- net N$1: track 1.65 -> 1.11 mm
