File: CurrentProbe/main.sch (EAGLE design)
At the start: 15 parts, among them CN1 USB, J1 v+, J2 v-, U1 LT1999CS8-50PBF, X1 SMA-142-0701-801/806

Commit message: a
Parts:
- removed CN1: USB, adafruit:USBMINIB
- added X2: MINI-USB_SHIELD5P4-32005-400, con-cypressindustries:MINI-USB_SHIELD5P4-32005-400
Connections:
- net GND: no longer CN1.GND
- net VCC: no longer CN1.VBUS
Changed lines of the file:
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@@
 </classes>
 <parts>
-<part name="CN1" library="adafruit" library_urn="urn:adsk.eagle:library:420" deviceset="USB" device="MINIB" package3d_urn="urn:adsk.eagle:package:6240633/1" value="USB"/>
 <part name="U1" library="LTC_By_element14_Batch_1" deviceset="LT1999CS8-50PBF" device=""/>
 <part name="C1" library="rcl" library_urn="urn:adsk.eagle:library:334" deviceset="C-US" device="C0805" package3d_urn="urn:adsk.eagle:package:23617/2" value="100n"/>
@@
 <part name="J1" library="SparkFun-Connectors" library_urn="urn:adsk.eagle:library:513" deviceset="BANANA_CONN" device="" package3d_urn="urn:adsk.eagle:package:38018/1" value="v+"/>
 <part name="J2" library="SparkFun-Connectors" library_urn="urn:adsk.eagle:library:513" deviceset="BANANA_CONN" device="" package3d_urn="urn:adsk.eagle:package:38018/1" value="v-"/>
+<part name="X2" library="con-cypressindustries" library_urn="urn:adsk.eagle:library:138" deviceset="MINI-USB_SHIELD5P4-" device="32005-400" package3d_urn="urn:adsk.eagle:package:6462/1"/>
 </parts>
 <sheets>
@@
 </plain>
 <instances>
-<instance part="CN1" gate="G$1" x="25.4" y="43.18" smashed="yes">
-<attribute name="NAME" x="15.24" y="51.816" size="1.27" layer="95"/>
-<attribute name="VALUE" x="15.24" y="33.02" size="1.27" layer="96"/>
-</instance>
 <instance part="U1" gate="A" x="91.44" y="45.72" smashed="yes">
 <attribute name="NAME" x="86.487" y="61.6966" size="2.0828" layer="95" ratio="10" rot="SR0"/>
@@
 <attribute name="VALUE" x="59.944" y="-3.048" size="1.778" layer="96" font="vector"/>
 </instance>
+<instance part="X2" gate="G$1" x="22.86" y="43.18" smashed="yes" rot="R180">
+<attribute name="NAME" x="25.4" y="31.75" size="1.778" layer="95" rot="R180"/>
+<attribute name="VALUE" x="12.7" y="50.8" size="1.778" layer="96" rot="R270"/>
+</instance>
 </instances>
 <busses>
@@
 <net name="VCC" class="0">
 <segment>
-<pinref part="CN1" gate="G$1" pin="VBUS"/>
 <wire x1="35.56" y1="48.26" x2="40.64" y2="48.26" width="0.1524" layer="91"/>
 <pinref part="P+4" gate="VCC" pin="VCC"/>
@@
 <net name="GND" class="0">
 <segment>
-<pinref part="CN1" gate="G$1" pin="GND"/>
 <wire x1="35.56" y1="38.1" x2="40.64" y2="38.1" width="0.1524" layer="91"/>
 <pinref part="GND2" gate="1" pin="GND"/>

Commit message: a
Connections:
- net GND: now also X2G$1.5, X2S.S1, X2S.S2, X2S.S3, X2S.S4
- net VCC: now also X2G$1.1
Other:
- moved on the sheet: X2
Changed lines of the file:
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@@
 <part name="J2" library="SparkFun-Connectors" library_urn="urn:adsk.eagle:library:513" deviceset="BANANA_CONN" device="" package3d_urn="urn:adsk.eagle:package:38018/1" value="v-"/>
 <part name="X2" library="con-cypressindustries" library_urn="urn:adsk.eagle:library:138" deviceset="MINI-USB_SHIELD5P4-" device="32005-400" package3d_urn="urn:adsk.eagle:package:6462/1"/>
+<part name="GND9" library="supply1" library_urn="urn:adsk.eagle:library:371" deviceset="GND" device=""/>
 </parts>
 <sheets>
@@
 <attribute name="VALUE" x="64.516" y="77.089" size="1.778" layer="96"/>
 </instance>
-<instance part="P+4" gate="VCC" x="40.64" y="50.8" smashed="yes">
-<attribute name="VALUE" x="38.1" y="48.26" size="1.778" layer="96" rot="R90"/>
-</instance>
-<instance part="GND2" gate="1" x="40.64" y="35.56" smashed="yes">
-<attribute name="VALUE" x="38.1" y="33.02" size="1.778" layer="96"/>
+<instance part="P+4" gate="VCC" x="7.62" y="50.8" smashed="yes">
+<attribute name="VALUE" x="5.08" y="48.26" size="1.778" layer="96" rot="R90"/>
+</instance>
+<instance part="GND2" gate="1" x="7.62" y="35.56" smashed="yes">
+<attribute name="VALUE" x="5.08" y="33.02" size="1.778" layer="96"/>
 </instance>
 <instance part="GND3" gate="1" x="60.96" y="27.94" smashed="yes">
@@
 <attribute name="VALUE" x="59.944" y="-3.048" size="1.778" layer="96" font="vector"/>
 </instance>
-<instance part="X2" gate="G$1" x="22.86" y="43.18" smashed="yes" rot="R180">
-<attribute name="NAME" x="25.4" y="31.75" size="1.778" layer="95" rot="R180"/>
-<attribute name="VALUE" x="12.7" y="50.8" size="1.778" layer="96" rot="R270"/>
+<instance part="X2" gate="G$1" x="20.32" y="43.18" smashed="yes">
+<attribute name="NAME" x="17.78" y="54.61" size="1.778" layer="95"/>
+<attribute name="VALUE" x="30.48" y="35.56" size="1.778" layer="96" rot="R90"/>
+</instance>
+<instance part="X2" gate="S" x="17.78" y="25.4" smashed="yes">
+<attribute name="NAME" x="25.4" y="22.86" size="1.778" layer="95"/>
+</instance>
+<instance part="GND9" gate="1" x="17.78" y="17.78" smashed="yes">
+<attribute name="VALUE" x="15.24" y="15.24" size="1.778" layer="96"/>
 </instance>
 </instances>
@@
 <net name="VCC" class="0">
 <segment>
-<wire x1="35.56" y1="48.26" x2="40.64" y2="48.26" width="0.1524" layer="91"/>
 <pinref part="P+4" gate="VCC" pin="VCC"/>
+<pinref part="X2" gate="G$1" pin="1"/>
+<wire x1="15.24" y1="48.26" x2="7.62" y2="48.26" width="0.1524" layer="91"/>
 </segment>
 <segment>
@@
 <net name="GND" class="0">
 <segment>
-<wire x1="35.56" y1="38.1" x2="40.64" y2="38.1" width="0.1524" layer="91"/>
+<wire x1="15.24" y1="38.1" x2="7.62" y2="38.1" width="0.1524" layer="91"/>
 <pinref part="GND2" gate="1" pin="GND"/>
+<pinref part="X2" gate="G$1" pin="5"/>
 </segment>
 <segment>
@@
 <pinref part="GND8" gate="1" pin="GND"/>
 </segment>
+<segment>
+<pinref part="X2" gate="S" pin="S1"/>
+<wire x1="15.24" y1="22.86" x2="15.24" y2="20.32" width="0.1524" layer="91"/>
+<pinref part="X2" gate="S" pin="S2"/>
+<wire x1="15.24" y1="20.32" x2="17.78" y2="20.32" width="0.1524" layer="91"/>
+<wire x1="17.78" y1="20.32" x2="17.78" y2="22.86" width="0.1524" layer="91"/>
+<pinref part="X2" gate="S" pin="S3"/>
+<wire x1="17.78" y1="20.32" x2="20.32" y2="20.32" width="0.1524" layer="91"/>
+<wire x1="20.32" y1="20.32" x2="20.32" y2="22.86" width="0.1524" layer="91"/>
+<junction x="17.78" y="20.32"/>
+<pinref part="X2" gate="S" pin="S4"/>
+<wire x1="20.32" y1="20.32" x2="22.86" y2="20.32" width="0.1524" layer="91"/>
+<wire x1="22.86" y1="20.32" x2="22.86" y2="22.86" width="0.1524" layer="91"/>
+<junction x="20.32" y="20.32"/>
+<pinref part="GND9" gate="1" pin="GND"/>
+</segment>
 </net>
