File: Atmega32U4/main.sch (EAGLE design)
At the start: 0 parts

Commit message: a
Parts:
- added C1, C2: 10p, rcl:C-USC0603
- added C3, C4, C5, C6, C7: 100n, rcl:C-USC0603
- added C8, C9: 1u, rcl:C-USC0805
- added Q1: 16MHz, crystal:CRYSTALHC49U-V
- added R1, R2: 22, rcl:R-US_R0603
- added SJ1: (no value), jumper:SJ2W
- added U1: ATMEGA32U4-AU, Microcontroller:ATMEGA32U4-AU
- added U2: LD1117S33TR, IC:LD1117S33TR
- added USB1: ST-USB-001G, OPL_Connector:MICRO-USB-SMD-B-WITHOUT-POST-W/P(ST-USB-001G)
Connections:
- new net !RESET: U1.!RESET
- new net (INT.6/AIN0)PE6: U1.(INT.6/AIN0)PE6
- new net (OC0B/SCL/INT0)PD0: U1.(OC0B/SCL/INT0)PD0
- new net (PCINT1/SCLK)PB1: U1.(PCINT1/SCLK)PB1
- new net (PCINT7/OC0A/OC1C/!RTS!)PB7: U1.(PCINT7/OC0A/OC1C/!RTS!)PB7
- new net (PDI/PCINT2/MOSI)PB2: U1.(PDI/PCINT2/MOSI)PB2
- new net (PDO/PCINT3/MISO)PB3: U1.(PDO/PCINT3/MISO)PB3
- new net (RXD1/INT2)PD2: U1.(RXD1/INT2)PD2
- new net (SDA/INT1)PD1: U1.(SDA/INT1)PD1
- new net (SS/PCINT0)PB0: U1.(SS/PCINT0)PB0
- new net (TXD1/INT3)PD3: U1.(TXD1/INT3)PD3
- new net (XCK1/!CTS!)PD5: U1.(XCK1/!CTS!)PD5
- new net AREF: U1.AREF
- new net D+: R1.2, U1.D+
- new net D-: R2.2, U1.D-
- new net DM: R2.1, USB1.DM
- new net DP: R1.1, USB1.DP
- new net GND: C1.2, C2.2, C3.2, C4.2, C5.2, C6.2, C7.2, C8.2, C9.2, U1.GND_15, U1.GND_23, U1.GND_35, U1.GND_43, U1.UGND, U2.ADJ/GND, USB1.GND@1, USB1.GND@2, USB1.GND@3, USB1.GND@4, USB1.GND@5
- new net N$1: C4.1, C9.1, SJ1.1, U2.4, U2.OUT
- new net PB4(PCINT4/ADC11): U1.PB4(PCINT4/ADC11)
- new net PB5(PCINT5/OC1!A/OC!4B/ADC: U1.PB5(PCINT5/OC1!A/OC!4B/ADC
- new net PB6(PCINT6/OC1B/OC4B/ADC: U1.PB6(PCINT6/OC1B/OC4B/ADC
- new net PC6(OC3A/!OC4!A: U1.PC6(OC3A/!OC4!A
- new net PC7(ICP3/CLK0/OC4A: U1.PC7(ICP3/CLK0/OC4A
- new net PD4(ICP1/ADC8): U1.PD4(ICP1/ADC8)
- new net PD6(T1/!OC4D!/ADC9): U1.PD6(T1/!OC4D!/ADC9)
- new net PD7(T0/OC4D/ADC10): U1.PD7(T0/OC4D/ADC10)
- new net PE2(!HWB!): U1.PE2(!HWB!)
- new net PF0(ADC0): U1.PF0(ADC0)
- new net PF1(ADC1): U1.PF1(ADC1)
- new net PF4(ADC4/TCK): U1.PF4(ADC4/TCK)
- new net PF5(ADC5/TMS): U1.PF5(ADC5/TMS)
- new net PF6(ADC6/TDO): U1.PF6(ADC6/TDO)
- new net PF7(ADC7/TDI): U1.PF7(ADC7/TDI)
- new net UCAP: U1.UCAP
- new net VBUS: U1.VBUS
- new net VCC: C5.1, C6.1, C7.1, SJ1.2, U1.AVCC_24, U1.AVCC_44, U1.VCC_14, U1.VCC_34
- new net VDD: C3.1, C8.1, SJ1.3, U1.UVCC, U2.IN, USB1.VCC
- new net XTAL1: C1.1, Q1.1, U1.XTAL1
- new net XTAL2: C2.1, Q1.2, U1.XTAL2
