File: Electronic Load/main.brd (EAGLE design)
At the start: 100 x 59 mm, 86 parts, among them IC1 MCP602SN, IC2 7805, J1 USB_MINI-B_SMT, J2 ICSP, Q1 16MHz, U1 328P, X1 SCREWTERM_5MM_4WAY

Commit message: a
Connections:
- net N$29 renamed VLOAD
Changed lines of the file:
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@@
 <?xml version="1.0" encoding="utf-8"?>
 <!DOCTYPE eagle SYSTEM "eagle.dtd">
-<eagle version="9.5.1">
+<eagle version="9.5.2">
 <drawing>
 <settings>
-<setting alwaysvectorfont="yes"/>
+<setting alwaysvectorfont="no"/>
 <setting verticaltext="up"/>
 </settings>
 <grid distance="0.25" unitdist="mm" unit="mm" style="dots" multiple="1" display="yes" altdistance="5" altunitdist="mil" altunit="mil"/>
 <layers>
-<layer number="1" name="Top" color="4" fill="1" visible="no" active="yes"/>
+<layer number="1" name="Top" color="4" fill="1" visible="yes" active="yes"/>
 <layer number="2" name="Route2" color="16" fill="1" visible="no" active="no"/>
 <layer number="3" name="Route3" color="17" fill="1" visible="no" active="no"/>
@@
 </signal>
 <signal name="RX">
-<contactref element="BR1" pad="5"/>
 <contactref element="U1" pad="3"/>
-<wire x1="55.5" y1="31.5" x2="65.5" y2="31.5" width="0.6096" layer="1"/>
+<wire x1="51" y1="31.5" x2="65.5" y2="31.5" width="0.6096" layer="1"/>
 <wire x1="65.5" y1="31.5" x2="66.5" y2="30.5" width="0.6096" layer="1"/>
 <via x="66.5" y="30.5" extent="1-16" drill="0.5" shape="octagon"/>
-<contactref element="SV1" pad="3"/>
-<wire x1="92" y1="21.27" x2="90.52" y2="22.75" width="0.6096" layer="16"/>
 <wire x1="66.5" y1="30.5" x2="66.5" y2="30" width="0.6096" layer="16"/>
-<wire x1="20.58" y1="33.92" x2="20.255" y2="33.92" width="0.6096" layer="1"/>
 <wire x1="20.58" y1="33.92" x2="23" y2="31.5" width="0.6096" layer="1"/>
 <wire x1="23" y1="31.5" x2="51" y2="31.5" width="0.6096" layer="1"/>
-<wire x1="51" y1="31.5" x2="55.5" y2="31.5" width="0.6096" layer="1"/>
 <wire x1="51.255" y1="35.27" x2="51.255" y2="31.755" width="0.6096" layer="1"/>
 <wire x1="51.255" y1="31.755" x2="51" y2="31.5" width="0.6096" layer="1"/>
-<wire x1="90.52" y1="22.75" x2="83.07763125" y2="22.75" width="0.6096" layer="16"/>
+<wire x1="83.07763125" y1="22.75" x2="90.52" y2="22.75" width="0.6096" layer="16"/>
 <wire x1="83.07763125" y1="22.75" x2="81.56563125" y2="24.262" width="0.6096" layer="16"/>
 <wire x1="72.238" y1="24.262" x2="81.56563125" y2="24.262" width="0.6096" layer="16"/>
 <wire x1="66.5" y1="30" x2="72.238" y2="24.262" width="0.6096" layer="16"/>
+<contactref element="SV1" pad="3"/>
+<contactref element="BR1" pad="5"/>
+<wire x1="90.52" y1="22.75" x2="92" y2="21.27" width="0.508" layer="16"/>
+<wire x1="20.255" y1="33.92" x2="20.58" y2="33.92" width="0.508" layer="1"/>
 </signal>
 <signal name="TX">
-<contactref element="BR1" pad="6"/>
 <contactref element="U1" pad="2"/>
-<contactref element="SV1" pad="5"/>
 <wire x1="53.795" y1="35.27" x2="53.795" y2="35.795" width="0.6096" layer="1"/>
 <wire x1="53.795" y1="35.795" x2="55.5" y2="37.5" width="0.6096" layer="1"/>
 <wire x1="55.5" y1="37.5" x2="58" y2="37.5" width="0.6096" layer="1"/>
-<wire x1="84.23" y1="21.27" x2="89.46" y2="21.27" width="0.6096" layer="1"/>
 <wire x1="58" y1="37.5" x2="61" y2="34.5" width="0.6096" layer="1"/>
 <wire x1="61" y1="34.5" x2="71" y2="34.5" width="0.6096" layer="1"/>
 <wire x1="71" y1="34.5" x2="84.23" y2="21.27" width="0.6096" layer="1"/>
-<wire x1="20.255" y1="36.46" x2="20.255" y2="36.245" width="0.6096" layer="1"/>
-<wire x1="20.255" y1="36.245" x2="22.5" y2="34" width="0.6096" layer="1"/>
-<wire x1="22.5" y1="34" x2="24" y2="32.5" width="0.6096" layer="1"/>
-<wire x1="24" y1="32.5" x2="30" y2="32.5" width="0.6096" layer="1"/>
-<wire x1="30" y1="32.5" x2="48" y2="32.5" width="0.6096" layer="1"/>
+<wire x1="20.255" y1="36.245" x2="24" y2="32.5" width="0.6096" layer="1"/>
+<wire x1="24" y1="32.5" x2="48" y2="32.5" width="0.6096" layer="1"/>
 <wire x1="48" y1="32.5" x2="48.5" y2="32.5" width="0.4064" layer="1"/>
 <wire x1="48.5" y1="32.5" x2="50" y2="34" width="0.4064" layer="1"/>
@@
 <wire x1="52.59" y1="37" x2="53.795" y2="35.795" width="0.4064" layer="1"/>
 <wire x1="50" y1="34" x2="50" y2="36.5" width="0.4064" layer="1"/>
+<contactref element="SV1" pad="5"/>
+<contactref element="BR1" pad="6"/>
+<wire x1="84.23" y1="21.27" x2="89.46" y2="21.27" width="0.508" layer="1"/>
+<wire x1="20.255" y1="36.46" x2="20.255" y2="36.245" width="0.508" layer="1"/>
 </signal>
 <signal name="V+">
@@
 <contactref element="U$1" pad="P$10"/>
 <contactref element="U$1" pad="P$11"/>
-<contactref element="U1" pad="27"/>
-<contactref element="R3" pad="1"/>
 <contactref element="U$3" pad="8"/>
 <wire x1="84.5" y1="39.05" x2="84.5" y2="38" width="0.3048" layer="16"/>
@@
 <wire x1="84.5" y1="39.05" x2="85" y2="39.05" width="0.3048" layer="16"/>
 <contactref element="SV1" pad="4"/>
-<wire x1="53.795" y1="27.65" x2="52.5" y2="28.945" width="0.6096" layer="16"/>
-<wire x1="52.5" y1="28.945" x2="52.5" y2="30.05" width="0.6096" layer="16"/>
 <wire x1="92" y1="18.73" x2="92" y2="18" width="0.6096" layer="16"/>
 <wire x1="92" y1="18" x2="90.7792" y2="16.7792" width="0.6096" layer="16"/>
@@
 <via x="62" y="28" extent="1-16" drill="0.5" shape="octagon"/>
 <wire x1="62" y1="28" x2="59.5" y2="25.5" width="0.6096" layer="1"/>
-<wire x1="55.945" y1="25.5" x2="53.795" y2="27.65" width="0.6096" layer="1"/>
 <wire x1="73" y1="39" x2="62" y2="28" width="0.6096" layer="16"/>
 <wire x1="59.5" y1="25.5" x2="55.945" y2="25.5" width="0.6096" layer="1"/>
-<wire x1="64.6658" y1="16.7792" x2="53.795" y2="27.65" width="0.6096" layer="16"/>
 <wire x1="90.7792" y1="16.7792" x2="64.6658" y2="16.7792" width="0.6096" layer="16"/>
+<contactref element="U1" pad="27"/>
+<contactref element="R3" pad="1"/>
+<wire x1="53.795" y1="27.65" x2="52.5" y2="28.945" width="0.6096" layer="16"/>
+<wire x1="52.5" y1="28.945" x2="52.5" y2="30.05" width="0.6096" layer="16"/>
+<wire x1="64.6658" y1="16.7792" x2="53.795" y2="27.65" width="0.508" layer="16"/>
+<wire x1="55.945" y1="25.5" x2="53.795" y2="27.65" width="0.508" layer="1"/>
 </signal>
 <signal name="SCL">
 <contactref element="U1" pad="28"/>
 <contactref element="R5" pad="1"/>
-<contactref element="U$1" pad="P$9"/>
 <contactref element="U$3" pad="7"/>
-<wire x1="84" y1="39.05" x2="84" y2="39.5" width="0.3048" layer="16"/>
 <wire x1="84" y1="39.5" x2="83.5" y2="40" width="0.3048" layer="16"/>
 <wire x1="74.685" y1="41.815" x2="72.875" y2="41.815" width="0.3048" layer="16"/>
@@
 <wire x1="81.5" y1="22.25" x2="64.9" y2="22.25" width="0.6096" layer="16"/>
 <wire x1="85.02" y1="18.73" x2="89.46" y2="18.73" width="0.6096" layer="16"/>
+<contactref element="U$1" pad="P$9"/>
+<wire x1="84" y1="39.05" x2="84" y2="39.5" width="0.254" layer="16"/>
 </signal>
 <signal name="SCK">
@@
 <contactref element="R17" pad="2"/>
 <contactref element="R18" pad="2"/>
-<contactref element="IC1" pad="3"/>
 <contactref element="IC1" pad="5"/>
 <wire x1="64.9" y1="46.595" x2="64.9" y2="45.05" width="0.508" layer="16"/>
@@
 <wire x1="65" y1="44.95" x2="65.05" y2="45" width="0.6096" layer="16"/>
 <wire x1="65.05" y1="45" x2="67.55" y2="45" width="0.6096" layer="16"/>
-<wire x1="70.1" y1="47.865" x2="68.185" y2="47.865" width="0.508" layer="16"/>
 <wire x1="67.55" y1="47.23" x2="67.55" y2="45" width="0.508" layer="16"/>
-<wire x1="68.185" y1="47.865" x2="67.55" y2="47.23" width="0.508" layer="16"/>
+<wire x1="67.55" y1="47.23" x2="68.185" y2="47.865" width="0.508" layer="16"/>
+<contactref element="IC1" pad="3"/>
+<wire x1="68.185" y1="47.865" x2="70.1" y2="47.865" width="0.508" layer="16"/>
 </signal>
 <signal name="N$20">
@@
 <wire x1="69.75" y1="57.45" x2="69.7" y2="57.5" width="0.508" layer="16"/>
 </signal>
-<signal name="N$29">
+<signal name="VLOAD">
 <contactref element="U$1" pad="P$16"/>
 <contactref element="R12" pad="2"/>
+<wire x1="86" y1="45.03" x2="85.5" y2="44.53" width="1.27" layer="1"/>
+<wire x1="87.5" y1="39.05" x2="88.5" y2="40.05" width="0.3048" layer="16"/>
+<wire x1="88.5" y1="40.05" x2="88.5" y2="44.5" width="0.3048" layer="16"/>
+<via x="88.5" y="44.5" extent="1-16" drill="0.5" shape="octagon"/>
+<wire x1="88.5" y1="44.5" x2="86.53" y2="44.5" width="0.3048" layer="1"/>
+<wire x1="86.53" y1="44.5" x2="86.265" y2="44.765" width="0.3048" layer="1"/>
 <contactref element="U$5" pad="D"/>
 <contactref element="U$4" pad="D"/>
@@
 <wire x1="64.77" y1="61.349" x2="84.066" y2="61.349" width="1.27" layer="1"/>
 <wire x1="84.066" y1="61.349" x2="86" y2="59.415" width="1.27" layer="1"/>
-<wire x1="86" y1="57.579" x2="86" y2="45.03" width="1.27" layer="1"/>
-<wire x1="86" y1="45.03" x2="85.5" y2="44.53" width="1.27" layer="1"/>
-<wire x1="87.5" y1="39.05" x2="88.5" y2="40.05" width="0.3048" layer="16"/>
-<wire x1="88.5" y1="40.05" x2="88.5" y2="44.5" width="0.3048" layer="16"/>
-<via x="88.5" y="44.5" extent="1-16" drill="0.5" shape="octagon"/>
-<wire x1="88.5" y1="44.5" x2="86.53" y2="44.5" width="0.3048" layer="1"/>
-<wire x1="86.53" y1="44.5" x2="86" y2="45.03" width="0.3048" layer="1"/>
+<wire x1="86" y1="57.579" x2="86" y2="45.03" width="1.016" layer="1"/>
+<wire x1="86" y1="45.03" x2="86.265" y2="44.765" width="1.016" layer="1"/>
 </signal>
 <signal name="VT">
