File: Electronic Load/main.sch (EAGLE design)
At the start: 86 parts, among them IC1 MCP602SN, IC2 7805, J1 USB_MINI-B_SMT, J2 ICSP, Q1 16MHz, U1 328P, X1 SCREWTERM_5MM_4WAY

Commit message: a
Connections:
- net N$29 renamed VLOAD
Other:
- note added: "Designed 03/2020"
- note added: "Electronic Load"
- note added: "Xavier Bourlot"
- note added: "increase part hole size"
- note added: "rev 1.0"
- moved on the sheet: C1, C11, C12, C13, C14, C15, C16, C17, C18, C19, C2, C20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
