File: ProgrammableFilter/dcdc.sch (EAGLE design)
At the start: 0 parts

Commit message: a
Parts:
- added C1: 330p, rcl:C-EUC0805
- added C2: 100u, rcl:CPOL-EUE5-10.5
- added C3, C4: 220u, rcl:CPOL-EUE5-10.5
- added C5, C6: 100n, rcl:C-EUC0805
- added D1: 1N5812, diode:1N5333
- added IC1: MC34063AP, mc34063:MC34063AP
- added R1: R2, rcl:R-EU_0207/10
- added R2: 1.5k, rcl:R-EU_R0805
- added R3: 13k, rcl:R-EU_R0805
- added R4: 0, rcl:R-EU_R0805
- added R5: 75, rcl:R-EU_0207/10
- added R6: R2, rcl:R-EU_R0805
- added R7: 75, rcl:R-EU_R0805
- added X1, X2: 22-23-2021, con-molex:22-23-2021
Connections:
- new net N$1: R3.2, R4.1
- new net N$2: R1.1, R6.1
- new net N$3: R1.2, R6.2
- new net N$4: R5.1, R7.1
- new net N$5: R5.2, R7.2
- new net N$6: IC1.GND, X1-2.S, X2-1.S
- new net N$7: IC1.VCC, X2-2.S
